Commit message: Gazebo integration

File: robots_description/Grippers/YumiServoGripper/yumi_servo_gripper.transmission.xacro (robot description, xacro)
@@ -4,8 +4,18 @@
     <transmission name="${name}_tran">
       <type>transmission_interface/SimpleTransmission</type>
-      <joint name="${name}_joint">
+      <joint name="gripper_joint_l">
         <hardwareInterface>${hardware_interface}</hardwareInterface>
       </joint>
-      <actuator name="${name}_motor">
+      <actuator name="${name}_motor_l">
+        <hardwareInterface>${hardware_interface}</hardwareInterface>
+        <mechanicalReduction>1</mechanicalReduction>
+      </actuator>
+    </transmission>
+    <transmission name="${name}_tran">
+      <type>transmission_interface/SimpleTransmission</type>
+      <joint name="gripper_joint_r">
+        <hardwareInterface>${hardware_interface}</hardwareInterface>
+      </joint>
+      <actuator name="${name}_motor_r">
         <hardwareInterface>${hardware_interface}</hardwareInterface>
         <mechanicalReduction>1</mechanicalReduction>

File: robots_description/Grippers/YumiServoGripper/yumi_servo_gripper.xacro (robot description, xacro)
@@ -1,10 +1,6 @@
 <?xml version="1.0"?>
 <robot name="yumi" xmlns:xacro="http://www.ros.org/wiki/xacro">
-   <!-- Import all Gazebo-customization elements, including Gazebo colors -->
-   <xacro:include
-      filename="$(find robots_description)/Grippers/YumiServoGripper/yumi_servo_gripper.gazebo.xacro" />
    <!-- Import Transmissions -->
-   <xacro:include
-      filename="$(find robots_description)/Grippers/YumiServoGripper/yumi_servo_gripper.transmission.xacro" />
+   <xacro:include filename="$(find robots_description)/Grippers/YumiServoGripper/yumi_servo_gripper.transmission.xacro" />
    <!-- some constants -->
    <xacro:property name="joint_damping" value="0.5" />
@@ -16,5 +12,5 @@
       between {parent} and base-->
       <joint name="${parent}_joint" type="fixed">
-         <xacro:insert_block name="origin" />
+         <origin xyz="0 0.0 0.0" rpy="0 0 0" />
          <parent link="${parent}" />
          <child link="${name}_base" />
@@ -31,5 +27,4 @@
                <mesh filename="package://robots_description/meshes/Yumi/gripper/base.stl" />
             </geometry>
-            <material name="Light_Grey" />
          </visual>
          <collision>
@@ -38,9 +33,14 @@
                <mesh filename="package://robots_description/meshes/Yumi/gripper/coarse/base.stl" />
             </geometry>
-            <material name="Light_Grey" />
          </collision>
       </link>
+      <link name="grasp_link" />
+      <joint name="grasp_joint" type="fixed">
+         <origin xyz="0 0.0 0.13" rpy="0 0 0" />
+         <child link="grasp_link" />
+         <parent link="${name}_base" />
+      </joint>
       <!-- joint between base and right finger -->
-      <joint name="${name}_joint" type="prismatic">
+      <joint name="${name}_joint_r" type="prismatic">
          <parent link="${name}_base" />
          <child link="${name}_finger_r" />
@@ -52,5 +52,9 @@
       </joint>
       <link name="${name}_finger_r">
-         <xacro:cuboid_inertia mass="0.04" width="0.05" height="0.05" length="0.05" />
+         <inertial>
+            <origin xyz="0 0 0" rpy="0 0 0" />
+            <mass value="0.1" />
+            <inertia ixx="0.01" ixy="0" ixz="0" iyy="0.01" iyz="0" izz="0.01" />
+         </inertial>
          <visual>
             <origin xyz="0 0 0" rpy="0 0 0" />
@@ -69,5 +73,5 @@
       </link>
       <!-- joint between base and left finger -->
-      <joint name="${name}_joint_m" type="prismatic">
+      <joint name="${name}_joint_l" type="prismatic">
          <parent link="${name}_base" />
          <child link="${name}_finger_l" />
@@ -77,8 +81,11 @@
             effort="${max_gripper_effort}" velocity="${max_gripper_velocity}" />
          <dynamics damping="${gripper_joint_damping}" />
-         <mimic joint="${name}_joint" />
       </joint>
       <link name="${name}_finger_l">
-         <xacro:cuboid_inertia mass="0.04" width="0.05" height="0.05" length="0.05" />
+         <inertial>
+            <origin xyz="0 0 0" rpy="0 0 0" />
+            <mass value="0.1" />
+            <inertia ixx="0.01" ixy="0" ixz="0" iyy="0.01" iyz="0" izz="0.01" />
+         </inertial>
          <visual>
             <origin xyz="0 0 0" rpy="0 0 0" />
@@ -97,6 +104,26 @@
       </link>
       <!--Extensions -->
-      <xacro:yumi_servo_gripper_gazebo name="SmartGripper" />
       <xacro:yumi_servo_gripper_transmission name="SmartGripper" hardware_interface="${hardware_interface}" />
+      <gazebo reference="${parent}_joint">
+         <disableFixedJointLumping>true</disableFixedJointLumping>
+         <preserveFixedJoint>true</preserveFixedJoint>
+      </gazebo>
+      <gazebo>
+         <plugin name="gazebo_grasp_fix" filename="libgazebo_grasp_fix.so">
+            <arm>
+               <arm_name>yumi</arm_name>
+               <palm_link>gripper_base</palm_link>
+               <gripper_link> gripper_finger_l </gripper_link>
+               <gripper_link> gripper_finger_r </gripper_link>
+            </arm>
+            <forces_angle_tolerance>100</forces_angle_tolerance>
+            <update_rate>4</update_rate>
+            <grip_count_threshold>4</grip_count_threshold>
+            <max_grip_count>8</max_grip_count>
+            <release_tolerance>0.005</release_tolerance>
+            <disable_collisions_on_attach>false</disable_collisions_on_attach>
+            <contact_topic>__default_topic__</contact_topic>
+         </plugin>
+      </gazebo>
    </xacro:macro>
 </robot>

File: robots_description/xacro/YumiSingleArm/single_yumi.transmission.xacro (robot description, xacro)
@@ -4,5 +4,5 @@
       <transmission name="${name}_tran_1">
          <type>transmission_interface/SimpleTransmission</type>
-         <joint name="${name}_joint_1">
+         <joint name="joint_1">
                <hardwareInterface>${hardware_interface}</hardwareInterface>
          </joint>
@@ -14,5 +14,5 @@
       <transmission name="${name}_tran_2">
          <type>transmission_interface/SimpleTransmission</type>
-         <joint name="${name}_joint_2">
+         <joint name="joint_2">
             <hardwareInterface>${hardware_interface}</hardwareInterface>
          </joint>
@@ -24,5 +24,5 @@
       <transmission name="${name}_tran_3">
          <type>transmission_interface/SimpleTransmission</type>
-         <joint name="${name}_joint_3">
+         <joint name="joint_3">
             <hardwareInterface>${hardware_interface}</hardwareInterface>
          </joint>
@@ -34,5 +34,5 @@
       <transmission name="${name}_tran_4">
          <type>transmission_interface/SimpleTransmission</type>
-         <joint name="${name}_joint_4">
+         <joint name="joint_4">
             <hardwareInterface>${hardware_interface}</hardwareInterface>
          </joint>
@@ -44,5 +44,5 @@
       <transmission name="${name}_tran_5">
          <type>transmission_interface/SimpleTransmission</type>
-         <joint name="${name}_joint_5">
+         <joint name="joint_5">
             <hardwareInterface>${hardware_interface}</hardwareInterface>
          </joint>
@@ -54,5 +54,5 @@
       <transmission name="${name}_tran_6">
          <type>transmission_interface/SimpleTransmission</type>
-         <joint name="${name}_joint_6">
+         <joint name="joint_6">
             <hardwareInterface>${hardware_interface}</hardwareInterface>
          </joint>
@@ -64,5 +64,5 @@
       <transmission name="${name}_tran_7">
          <type>transmission_interface/SimpleTransmission</type>
-         <joint name="${name}_joint_7">
+         <joint name="joint_7">
             <hardwareInterface>${hardware_interface}</hardwareInterface>
          </joint>

File: robots_description/xacro/YumiSingleArm/single_yumi.xacro (robot description, xacro)
@@ -1,6 +1,4 @@
 <?xml version="1.0"?>
 <robot name="single_yumi" xmlns:xacro="http://www.ros.org/wiki/xacro">
-  <!-- Import all Gazebo-customization elements, including Gazebo colors -->
-  <xacro:include filename="$(find robots_description)/xacro/YumiSingleArm/single_yumi.gazebo.xacro" />
   <!-- Import Transmissions -->
   <xacro:include filename="$(find robots_description)/xacro/YumiSingleArm/single_yumi.transmission.xacro" />
@@ -16,4 +14,9 @@
     </joint>
     <link name="single_yumi_base_link">
+      <inertial>
+        <origin xyz="0 -0.03 0.12" rpy="0 0 0" />
+        <mass value="2" />
+        <inertia ixx="0.1" ixy="0" ixz="0" iyy="0.1" iyz="0" izz="0.1" />
+      </inertial>
       <visual>
         <origin xyz="0 0 0" rpy="0 0 0" />
@@ -23,4 +26,11 @@
         <material name="Grey" />
       </visual>
+      <collision>
+        <origin xyz="0 0 0" rpy="0 0 0" />
+        <geometry>
+          <mesh filename="package://robots_description/meshes/Yumi/coarse/single_arm_base.stl" />
+        </geometry>
+        <material name="Grey" />
+      </collision>
     </link>
     <!-- joint between body and link_1 -->
@@ -242,5 +252,4 @@
     </link>
     <!--Extensions -->
-    <xacro:single_yumi_gazebo name="single_arm" />
     <xacro:single_yumi_transmission name="single_arm" hardware_interface="${hardware_interface}"/>
   </xacro:macro>
