Commit message: Fixed namespace name + joint finger in simulation

File: robots_description/Grippers/YumiServoGripper/yumi_servo_gripper.xacro (robot description, xacro)
@@ -8,5 +8,7 @@
    <xacro:property name="max_gripper_effort" value="20" />
    <xacro:property name="max_gripper_velocity" value="2" />
-   <xacro:macro name="yumi_servo_gripper" params="parent name hardware_interface *origin">
+   <xacro:macro name="yumi_servo_gripper" params="parent name hardware_interface fake_execution *origin">
+      <xacro:arg name="fake_execution"     default="$(arg fake_execution)" />
+      <xacro:property name="fake_execution"     value="$(arg fake_execution)" />
       <!--joint
       between {parent} and base-->
@@ -41,89 +43,91 @@
          <parent link="${name}_base" />
       </joint>
-      <!-- joint between base and right finger -->
-      <joint name="${name}_joint_r" type="prismatic">
-         <parent link="${name}_base" />
-         <child link="${name}_finger_r" />
-         <origin xyz="0 -0.0065 0.0837" rpy="0 0 0" />
-         <axis xyz="-1 0 0" />
-         <limit lower="0" upper="0.025"
-            effort="${max_gripper_effort}" velocity="${max_gripper_velocity}" />
-         <dynamics damping="${gripper_joint_damping}" />
-      </joint>
-      <link name="${name}_finger_r">
-         <inertial>
-            <origin xyz="0 0 0" rpy="0 0 0" />
-            <mass value="0.1" />
-            <inertia ixx="0.01" ixy="0" ixz="0" iyy="0.01" iyz="0" izz="0.01" />
-         </inertial>
-         <visual>
-            <origin xyz="0 0 0" rpy="0 0 0" />
-            <geometry>
-               <mesh filename="package://robots_description/meshes/Yumi/gripper/finger.stl" />
-            </geometry>
-            <material name="Blue" />
-         </visual>
-         <collision>
-            <origin xyz="0 0 0" rpy="0 0 0" />
-            <geometry>
-               <mesh filename="package://robots_description/meshes/Yumi/gripper/coarse/finger.stl" />
-            </geometry>
-            <material name="Blue" />
-         </collision>
-      </link>
-      <!-- joint between base and left finger -->
-      <joint name="${name}_joint_l" type="prismatic">
-         <parent link="${name}_base" />
-         <child link="${name}_finger_l" />
-         <origin xyz="0 0.0065 0.0837" rpy="0 0 ${PI}" />
-         <axis xyz="-1 0 0" />
-         <limit lower="0" upper="0.025"
-            effort="${max_gripper_effort}" velocity="${max_gripper_velocity}" />
-         <dynamics damping="${gripper_joint_damping}" />
-      </joint>
-      <link name="${name}_finger_l">
-         <inertial>
-            <origin xyz="0 0 0" rpy="0 0 0" />
-            <mass value="0.1" />
-            <inertia ixx="0.01" ixy="0" ixz="0" iyy="0.01" iyz="0" izz="0.01" />
-         </inertial>
-         <visual>
-            <origin xyz="0 0 0" rpy="0 0 0" />
-            <geometry>
-               <mesh filename="package://robots_description/meshes/Yumi/gripper/finger.stl" />
-            </geometry>
-            <material name="Blue" />
-         </visual>
-         <collision>
-            <origin xyz="0 0 0" rpy="0 0 0" />
-            <geometry>
-               <mesh filename="package://robots_description/meshes/Yumi/gripper/coarse/finger.stl" />
-            </geometry>
-            <material name="Blue" />
-         </collision>
-      </link>
-      <!--Extensions -->
-      <xacro:yumi_servo_gripper_transmission name="SmartGripper" hardware_interface="${hardware_interface}" />
-      <gazebo reference="${parent}_joint">
-         <disableFixedJointLumping>true</disableFixedJointLumping>
-         <preserveFixedJoint>true</preserveFixedJoint>
-      </gazebo>
-      <gazebo>
-         <plugin name="gazebo_grasp_fix" filename="libgazebo_grasp_fix.so">
-            <arm>
-               <arm_name>yumi</arm_name>
-               <palm_link>gripper_base</palm_link>
-               <gripper_link> gripper_finger_l </gripper_link>
-               <gripper_link> gripper_finger_r </gripper_link>
-            </arm>
-            <forces_angle_tolerance>100</forces_angle_tolerance>
-            <update_rate>4</update_rate>
-            <grip_count_threshold>4</grip_count_threshold>
-            <max_grip_count>8</max_grip_count>
-            <release_tolerance>0.005</release_tolerance>
-            <disable_collisions_on_attach>false</disable_collisions_on_attach>
-            <contact_topic>__default_topic__</contact_topic>
-         </plugin>
-      </gazebo>
+      <xacro:if value="${fake_execution == 'true'}">
+         <!-- joint between base and right finger -->
+         <joint name="${name}_joint_r" type="prismatic">
+            <parent link="${name}_base" />
+            <child link="${name}_finger_r" />
+            <origin xyz="0 -0.0065 0.0837" rpy="0 0 0" />
+            <axis xyz="-1 0 0" />
+            <limit lower="0" upper="0.025"
+               effort="${max_gripper_effort}" velocity="${max_gripper_velocity}" />
+            <dynamics damping="${gripper_joint_damping}" />
+         </joint>
+         <link name="${name}_finger_r">
+            <inertial>
+               <origin xyz="0 0 0" rpy="0 0 0" />
+               <mass value="0.1" />
+               <inertia ixx="0.01" ixy="0" ixz="0" iyy="0.01" iyz="0" izz="0.01" />
+            </inertial>
+            <visual>
+               <origin xyz="0 0 0" rpy="0 0 0" />
+               <geometry>
+                  <mesh filename="package://robots_description/meshes/Yumi/gripper/finger.stl" />
+               </geometry>
+               <material name="Blue" />
+            </visual>
+            <collision>
+               <origin xyz="0 0 0" rpy="0 0 0" />
+               <geometry>
+                  <mesh filename="package://robots_description/meshes/Yumi/gripper/coarse/finger.stl" />
+               </geometry>
+               <material name="Blue" />
+            </collision>
+         </link>
+         <!-- joint between base and left finger -->
+         <joint name="${name}_joint_l" type="prismatic">
+            <parent link="${name}_base" />
+            <child link="${name}_finger_l" />
+            <origin xyz="0 0.0065 0.0837" rpy="0 0 ${PI}" />
+            <axis xyz="-1 0 0" />
+            <limit lower="0" upper="0.025"
+               effort="${max_gripper_effort}" velocity="${max_gripper_velocity}" />
+            <dynamics damping="${gripper_joint_damping}" />
+         </joint>
+         <link name="${name}_finger_l">
+            <inertial>
+               <origin xyz="0 0 0" rpy="0 0 0" />
+               <mass value="0.1" />
+               <inertia ixx="0.01" ixy="0" ixz="0" iyy="0.01" iyz="0" izz="0.01" />
+            </inertial>
+            <visual>
+               <origin xyz="0 0 0" rpy="0 0 0" />
+               <geometry>
+                  <mesh filename="package://robots_description/meshes/Yumi/gripper/finger.stl" />
+               </geometry>
+               <material name="Blue" />
+            </visual>
+            <collision>
+               <origin xyz="0 0 0" rpy="0 0 0" />
+               <geometry>
+                  <mesh filename="package://robots_description/meshes/Yumi/gripper/coarse/finger.stl" />
+               </geometry>
+               <material name="Blue" />
+            </collision>
+         </link>
+         <!--Extensions -->
+         <xacro:yumi_servo_gripper_transmission name="SmartGripper" hardware_interface="${hardware_interface}" />
+         <gazebo reference="${parent}_joint">
+            <disableFixedJointLumping>true</disableFixedJointLumping>
+            <preserveFixedJoint>true</preserveFixedJoint>
+         </gazebo>
+         <gazebo>
+            <plugin name="gazebo_grasp_fix" filename="libgazebo_grasp_fix.so">
+               <arm>
+                  <arm_name>yumi</arm_name>
+                  <palm_link>gripper_base</palm_link>
+                  <gripper_link> gripper_finger_l </gripper_link>
+                  <gripper_link> gripper_finger_r </gripper_link>
+               </arm>
+               <forces_angle_tolerance>100</forces_angle_tolerance>
+               <update_rate>4</update_rate>
+               <grip_count_threshold>4</grip_count_threshold>
+               <max_grip_count>8</max_grip_count>
+               <release_tolerance>0.005</release_tolerance>
+               <disable_collisions_on_attach>false</disable_collisions_on_attach>
+               <contact_topic>__default_topic__</contact_topic>
+            </plugin>
+         </gazebo>
+      </xacro:if>
    </xacro:macro>
 </robot>

File: robots_description/xacro/robot.urdf.xacro (robot description, xacro)
@@ -3,9 +3,12 @@
     <!-- Parameters -->
     <arg name="name"                     default="gofa" />
+    <arg name="fake_execution"           default="false" />
     <xacro:arg name="robot"              default="$(arg name)" />
+    <xacro:arg name="fake_execution"     default="$(arg fake_execution)" />
     <xacro:arg name="hardware_interface" default="PositionJointInterface" />
     <xacro:arg name="gripper_interface"  default="EffortJointInterface" />
     <xacro:arg name="yumi_setup"         default="default" />
     <xacro:property name="robot"              value="$(arg robot)" />
+    <xacro:property name="fake_execution"     value="$(arg fake_execution)" />
     <xacro:property name="hardware_interface" value="$(arg hardware_interface)" />
     <xacro:property name="gripper_interface"  value="$(arg gripper_interface)" />
@@ -35,5 +38,5 @@
         </xacro:single_yumi>
         <!-- Gripper -->
-        <xacro:yumi_servo_gripper name="gripper" parent="link_7" hardware_interface="${gripper_interface}">
+        <xacro:yumi_servo_gripper name="gripper" parent="link_7" hardware_interface="${gripper_interface}" fake_execution="${fake_execution}">
             <origin xyz="0 0 0.007" rpy="0 0 ${PI}" />
         </xacro:yumi_servo_gripper>

Commit message: Fix 2.0

File: robots_description/Grippers/YumiServoGripper/yumi_servo_gripper.xacro (robot description, xacro)
@@ -8,7 +8,5 @@
    <xacro:property name="max_gripper_effort" value="20" />
    <xacro:property name="max_gripper_velocity" value="2" />
-   <xacro:macro name="yumi_servo_gripper" params="parent name hardware_interface fake_execution *origin">
-      <xacro:arg name="fake_execution"     default="$(arg fake_execution)" />
-      <xacro:property name="fake_execution"     value="$(arg fake_execution)" />
+   <xacro:macro name="yumi_servo_gripper" params="parent name hardware_interface fake_execution:=true *origin">
       <!--joint
       between {parent} and base-->
