Commit message: irim_ss_pkg fixes

File: irim_ss_pkg/xacro/Extra/camera_stand.xacro (robot description, xacro)
@@ -2,6 +2,6 @@
 <robot name="camera_stand" xmlns:xacro="http://www.ros.org/wiki/xacro">
     <xacro:macro name="camera_stand" params="parent *origin">
-        <xacro:property name="base_height" value="0.6" />
-        <xacro:property name="holder_length" value="0.4" />
+        <xacro:property name="base_height" value="0.88" />
+        <xacro:property name="holder_length" value="0.3" />
         <joint name="joint_camera_stand_robot" type="fixed">
             <xacro:insert_block name="origin"/>
@@ -18,5 +18,5 @@
                 <origin xyz="0 0 ${base_height/2}" rpy="0 0 0"/>
                 <geometry>
-                    <box size="0.1 0.1 ${base_height}" />
+                    <box size="0.04 0.04 ${base_height}" />
                 </geometry>
             </visual>
@@ -24,5 +24,5 @@
                 <origin xyz="0 0 ${base_height/2}" rpy="0 0 0"/>
                 <geometry>
-                    <box size="0.1 0.1 ${base_height}" />
+                    <box size="0.04 0.04 ${base_height}" />
                 </geometry>
             </collision>
@@ -37,5 +37,5 @@
                 <origin xyz="0 0 ${holder_length/2}" rpy="0 0 0"/>
                 <geometry>
-                    <box size="0.1 0.1 ${holder_length}" />
+                    <box size="0.04 0.04 ${holder_length}" />
                 </geometry>
             </visual>
@@ -48,5 +48,5 @@
         </link>
         <joint name="joint_camera_holder" type="fixed">
-            <origin xyz="0.0 0.0 ${base_height}" rpy="0.0 -${pi/2} 0" />
+            <origin xyz="0.0 0.0 ${base_height}" rpy="${pi/2} -${pi/2} 0" />
             <parent link="base_link_camera_stand" />
             <child link="camera_holder" />
@@ -67,5 +67,5 @@
         </link>
         <joint name="joint_camera_link" type="fixed">
-            <origin xyz="0.0 0.0 ${holder_length + 0.1}" rpy="-${pi/2} 0 -2.5 " />
+            <origin xyz="0.0 0.0 ${holder_length + 0.1}" rpy="-${pi/2} 0 -3.14 " />
             <parent link="camera_holder" />
             <child link="ext_camera_link" />
@@ -75,5 +75,5 @@
             <update_rate>5.0</update_rate>
             <camera name="head">
-                <horizontal_fov>1.3962634</horizontal_fov>
+                <horizontal_fov>1.01</horizontal_fov>
                 <image>
                     <width>1280</width>
@@ -98,7 +98,7 @@
                 <updateRate>5.0</updateRate>
                 <cameraName>camera</cameraName>
-                <imageTopicName>image_raw</imageTopicName>
+                <imageTopicName>/oak/rgb/image_raw</imageTopicName>
                 <cameraInfoTopicName>camera_info</cameraInfoTopicName>
-                <frameName>camerext_camera_linka_link</frameName>
+                <frameName>ext_camera_link</frameName>
                 <!-- <hackBaseline>0.07</hackBaseline> -->
                 <distortionK1>0.000001</distortionK1>

File: irim_ss_pkg/xacro/Extra/table.xacro (robot description, xacro)
@@ -11,5 +11,5 @@
         </joint>
         <gazebo reference="base_link_table">
-            <material>Gazebo/Yellow</material>
+            <material>Gazebo/Grey</material>
         </gazebo>
         <link name="base_link_table">
@@ -77,3 +77,7 @@
         </link>
     </xacro:macro>
+    <gazebo reference="base_link_table">
+        <mu1>0.2</mu1>
+        <mu2>0.1</mu2>
+    </gazebo>
 </robot>

File: irim_ss_pkg/xacro/irim_yumi.urdf.xacro (robot description, xacro)
@@ -4,4 +4,5 @@
     <xacro:arg name="hardware_interface" default="hardware_interface/PositionJointInterface" />
     <xacro:arg name="gripper_interface"  default="hardware_interface/EffortJointInterface" />
+    <!-- <xacro:arg name="gripper_interface" default="hardware_interface/PositionJointInterface" /> -->
     <xacro:property name="robot"              value="yumi" />
     <xacro:property name="hardware_interface" value="$(arg hardware_interface)" />
@@ -22,10 +23,15 @@
     <xacro:include filename="$(find irim_ss_pkg)/xacro/Extra/camera_stand.xacro" />
     <xacro:camera_stand parent="base_link_table" >
-        <origin xyz="0.6 0.5 0.65" rpy="0 0 0" />
+        <origin xyz="0.0 0.4 0.65" rpy="0 0 0" />
     </xacro:camera_stand>
+    <!-- Import the surface -->
+    <xacro:include filename="$(find irim_ss_pkg)/xacro/Extra/surface.xacro" />
+    <xacro:surface parent="single_yumi_base_link" >
+        <origin xyz="-0.03 0.33 0.08" rpy="0 0 0" />
+    </xacro:surface>
     <!--Import the single yumi macro -->
     <xacro:include filename="$(find robots_description)/xacro/YumiSingleArm/single_yumi.xacro" />
     <xacro:single_yumi parent="base_link_table" hardware_interface="${hardware_interface}">
-        <origin xyz="-0.3 0 0.6" rpy="0 0 0" />
+        <origin xyz="-0.3 0 0.6" rpy="0 0 -1.57" />
     </xacro:single_yumi>
     <!--Import the yumi servo gripper macro -->

File: robots_description/Grippers/YumiServoGripper/yumi_servo_gripper.xacro (robot description, xacro)
@@ -122,5 +122,5 @@
                <grip_count_threshold>4</grip_count_threshold>
                <max_grip_count>8</max_grip_count>
-               <release_tolerance>0.005</release_tolerance>
+               <release_tolerance>0.002</release_tolerance>
                <disable_collisions_on_attach>false</disable_collisions_on_attach>
                <contact_topic>__default_topic__</contact_topic>
