Commit message: Fixed joint6 limit

File: moveit_config/gofa_moveit_config/config/gazebo_robot.urdf (robot description, URDF)
Before this commit: robot robot, 9 links, 8 joints
Joints:
- joint J6: limit lower=-3.141592653589793 upper=3.141592653589793 effort=0 velocity=3.490658503988659 -> lower=-4,71239 upper=4,71239 effort=0 velocity=3.490658503988659

File: robots_description/xacro/Gofa/gofa.urdf.xacro (robot description, xacro)
@@ -147,5 +147,5 @@
 			<child link="$(arg 6th_link_name)"/>
 			<axis xyz="1 0 0"/>
-			<limit effort="0" lower="${radians(-180)}" upper="${radians(180)}" velocity="${radians(200)}"/>
+			<limit effort="0" lower="${radians(-270)}" upper="${radians(270)}" velocity="${radians(200)}"/>
 		</joint>
 		<!-- Flange -->
