Commit message: Reverted

File: robots_description/xacro/YumiSingleArm/single_yumi.xacro (robot description, xacro)
@@ -1,247 +1,497 @@
 <?xml version="1.0"?>
 <robot name="single_yumi" xmlns:xacro="http://www.ros.org/wiki/xacro">
+<<<<<<< HEAD
 <!-- Import all Gazebo-customization elements, including Gazebo colors -->
 <xacro:include filename="$(find robots_description)/xacro/YumiSingleArm/single_yumi.gazebo.xacro" />
 <!-- Import Transmissions -->
 <xacro:include filename="$(find robots_description)/xacro/YumiSingleArm/single_yumi.transmission.xacro" />
-<!-- some constants -->
-<xacro:property name="joint_damping" value="0.5" />
-<xacro:property name="max_effort" value="300" />
+   <!-- some constants -->
+   <xacro:property name="joint_damping" value="0.5" />
+   <xacro:property name="max_effort" value="300" />
 <xacro:macro name="single_yumi" params="parent hardware_interface *origin">
-  <!-- joint between external and base -->
-  <joint name="joint_0" type="fixed">
-     <xacro:insert_block name="origin" />
-     <parent link="${parent}" />
-     <child link="single_yumi_base_link" />
-  </joint>
-  <link name="single_yumi_base_link">
-     <visual>
-        <origin xyz="0 0 0" rpy="0 0 0" />
-        <geometry>
-           <mesh filename="package://robots_description/meshes/Yumi/single_arm_base.stl" />
-        </geometry>
-        <material name="Grey" />
-     </visual>
-  </link>
-  <!-- joint between body and link_1 -->
-  <joint name="joint_1" type="revolute">
-     <parent link="single_yumi_base_link" />
-     <child link="link_1" />
-     <origin xyz="0.0 0.0 0.2048" rpy="0.0 0.0 ${PI}" />
-     <axis xyz="0 0 1" />
-     <limit lower="${-168.5 * PI / 180}" upper="${168.5 * PI / 180}"
+  <xacro:macro name="single_yumi" params="parent hardware_interface *origin">
+      <!-- joint between external and base -->
+      <joint name="joint_0" type="fixed">
+         <xacro:insert_block name="origin" />
+         <parent link="${parent}" />
+         <child link="single_yumi_base_link" />
+      </joint>
+      <link name="single_yumi_base_link">
+         <visual>
+            <origin xyz="0 0 0" rpy="0 0 0" />
+            <geometry>
+               <mesh filename="package://robots_description/meshes/Yumi/single_arm_base.stl" />
+            </geometry>
+            <material name="Grey" />
+         </visual>
+      </link>
+      <!-- joint between body and link_1 -->
+      <joint name="joint_1" type="revolute">
+         <parent link="single_yumi_base_link" />
+         <child link="link_1" />
+         <origin xyz="0.0 0.0 0.2048" rpy="0.0 0.0 ${PI}" />
+         <axis xyz="0 0 1" />
+         <limit lower="${-168.5 * PI / 180}" upper="${168.5 * PI / 180}"
+            effort="${max_effort}" velocity="${180 * PI / 180}" />
+         <dynamics damping="${joint_damping}" />
+      </joint>
+      <link name="link_1">
+         <inertial>
+            <origin xyz="0 -0.03 0.12" rpy="0 0 0" />
+            <mass value="2" />
+            <inertia ixx="0.1" ixy="0" ixz="0" iyy="0.1" iyz="0" izz="0.1" />
+         </inertial>
+         <visual>
+            <origin xyz="0 0 0" rpy="0 0 0" />
+            <geometry>
+               <mesh filename="package://robots_description/meshes/Yumi/link_1.stl" />
+            </geometry>
+            <material name="Grey" />
+         </visual>
+         <collision>
+            <origin xyz="0 0 0" rpy="0 0 0" />
+            <geometry>
+               <mesh filename="package://robots_description/meshes/Yumi/coarse/link_1.stl" />
+            </geometry>
+            <material name="Grey" />
+         </collision>
+      </link>
+      <!-- joint between link_1 and link_2 -->
+      <joint name="joint_2" type="revolute">
+         <parent link="link_1" />
+         <child link="link_2" />
+         <origin xyz="0.03 0.0 0.1" rpy="${PI / 2} 0.0 0.0" />
+         <axis xyz="0 0 1" />
+         <limit lower="${-143.5 * PI / 180}" upper="${43.5 * PI / 180}"
+            effort="${max_effort}" velocity="${180 * PI / 180}" />
+         <dynamics damping="${joint_damping}" />
+      </joint>
+      <link name="link_2">
+         <inertial>
+            <origin xyz="0 0 0" rpy="0 0 0" />
+            <mass value="2" />
+            <inertia ixx="0.1" ixy="0" ixz="0" iyy="0.1" iyz="0" izz="0.1" />
+         </inertial>
+         <visual>
+            <origin xyz="0 0 0" rpy="0 0 0" />
+            <geometry>
+               <mesh filename="package://robots_description/meshes/Yumi/link_2.stl" />
+            </geometry>
+            <material name="Grey" />
+         </visual>
+         <collision>
+            <origin xyz="0 0 0" rpy="0 0 0" />
+            <geometry>
+               <mesh filename="package://robots_description/meshes/Yumi/coarse/link_2.stl" />
+            </geometry>
+            <material name="Grey" />
+         </collision>
+      </link>
+      <!-- joint between link_2 and link_3 -->
+      <joint name="joint_3" type="revolute">
+         <parent link="link_2" />
+         <child link="link_3" />
+         <origin xyz="-0.03 0.17283 0.0" rpy="${-PI / 2} 0.0 0.0" />
+         <axis xyz="0 0 1" />
+         <limit lower="${-168.5 * PI / 180}" upper="${168.5 * PI / 180}"
+            effort="${max_effort}" velocity="${180 * PI / 180}" />
+         <dynamics damping="${joint_damping}" />
+      </joint>
+      <link name="link_3">
+         <inertial>
+            <origin xyz="0 0 0" rpy="0 0 0" />
+            <mass value="2" />
+            <inertia ixx="0.1" ixy="0" ixz="0" iyy="0.1" iyz="0" izz="0.1" />
+         </inertial>
+         <visual>
+            <origin xyz="0 0 0" rpy="0 0 0" />
+            <geometry>
+               <mesh filename="package://robots_description/meshes/Yumi/link_3.stl" />
+            </geometry>
+            <material name="Grey" />
+         </visual>
+         <collision>
+            <origin xyz="0 0 0" rpy="0 0 0" />
+            <geometry>
+               <mesh filename="package://robots_description/meshes/Yumi/coarse/link_3.stl" />
+            </geometry>
+            <material name="Grey" />
+         </collision>
+      </link>
+      <!-- joint between link_3 and link_4 -->
+      <joint name="joint_4" type="revolute">
+         <parent link="link_3" />
+         <child link="link_4" />
+         <origin xyz="-0.04188 0.0 0.07873" rpy="${PI / 2} ${- PI / 2} 0.0" />
+         <axis xyz="0 0 1" />
+         <limit lower="${-123.5 * PI / 180}" upper="${80 * PI / 180}"
+            effort="${max_effort}" velocity="${180 * PI / 180}" />
+         <dynamics damping="${joint_damping}" />
+      </joint>
+      <link name="link_4">
+         <inertial>
+            <origin xyz="0 0 0" rpy="0 0 0" />
+            <mass value="2" />
+            <inertia ixx="0.1" ixy="0" ixz="0" iyy="0.1" iyz="0" izz="0.1" />
+         </inertial>
+         <visual>
+            <origin xyz="0 0 0" rpy="0 0 0" />
+            <geometry>
+               <mesh filename="package://robots_description/meshes/Yumi/link_4.stl" />
+            </geometry>
+            <material name="Grey" />
+         </visual>
+         <collision>
+            <origin xyz="0 0 0" rpy="0 0 0" />
+            <geometry>
+               <mesh filename="package://robots_description/meshes/Yumi/coarse/link_4.stl" />
+            </geometry>
+            <material name="Grey" />
+         </collision>
+      </link>
+      <!-- joint between link_4 and link_5 -->
+      <joint name="joint_5" type="revolute">
+         <parent link="link_4" />
+         <child link="link_5" />
+         <origin xyz="0.0405 0.16461 0.0" rpy="-${PI / 2} 0.0 0.0" />
+         <axis xyz="0 0 1" />
+         <limit lower="${-290 * PI / 180}" upper="${290 * PI / 180}"
+            effort="${max_effort}" velocity="${400 * PI / 180}" />
+         <dynamics damping="${joint_damping}" />
+      </joint>
+      <link name="link_5">
+         <inertial>
+            <origin xyz="0 0 0" rpy="0 0 0" />
+            <mass value="2" />
+            <inertia ixx="0.1" ixy="0" ixz="0" iyy="0.1" iyz="0" izz="0.1" />
+         </inertial>
+         <visual>
+            <origin xyz="0 0 0" rpy="0 0 0" />
+            <geometry>
+               <mesh filename="package://robots_description/meshes/Yumi/link_5.stl" />
+            </geometry>
+            <material name="Grey" />
+         </visual>
+         <collision>
+            <origin xyz="0 0 0" rpy="0 0 0" />
+            <geometry>
+               <mesh filename="package://robots_description/meshes/Yumi/coarse/link_5.stl" />
+            </geometry>
+            <material name="Grey" />
+         </collision>
+      </link>
+      <!-- joint between link_5 and link_6 -->
+      <joint name="joint_6" type="revolute">
+         <parent link="link_5" />
+         <child link="link_6" />
+         <origin xyz="-0.027 0 0.10039" rpy="${PI / 2} 0.0 0.0" />
+         <axis xyz="0 0 1" />
+         <limit lower="${-88 * PI / 180}" upper="${138 * PI / 180}"
+            effort="${max_effort}" velocity="${400 * PI / 180}" />
+         <dynamics damping="${joint_damping}" />
+      </joint>
+      <link name="link_6">
+         <inertial>
+            <origin xyz="0 0 0" rpy="0 0 0" />
+            <mass value="2" />
+            <inertia ixx="0.1" ixy="0" ixz="0" iyy="0.1" iyz="0" izz="0.1" />
+         </inertial>
+         <visual>
+            <origin xyz="0 0 0" rpy="0 0 0" />
+            <geometry>
+               <mesh filename="package://robots_description/meshes/Yumi/link_6.stl" />
+            </geometry>
+            <material name="Grey" />
+         </visual>
+         <collision>
+            <origin xyz="0 0 0" rpy="0 0 0" />
+            <geometry>
+               <mesh filename="package://robots_description/meshes/Yumi/coarse/link_6.stl" />
+            </geometry>
+            <material name="Grey" />
+         </collision>
+      </link>
+      <!-- joint between link_6 and link_7 -->
+      <joint name="joint_7" type="revolute">
+         <parent link="link_6" />
+         <child link="link_7" />
+         <origin xyz="0.027 0.029 0.0" rpy="-${PI / 2} 0.0 0.0" />
+         <axis xyz="0 0 1" />
+         <limit lower="${-229 * PI / 180}" upper="${229 * PI / 180}"
+            effort="${max_effort}" velocity="${400 * PI / 180}" />
+         <dynamics damping="${joint_damping}" />
+      </joint>
+      <link name="link_7">
+         <inertial>
+            <origin xyz="0 0 0" rpy="0 0 0" />
+            <mass value="2" />
+            <inertia ixx="0.1" ixy="0" ixz="0" iyy="0.1" iyz="0" izz="0.1" />
+         </inertial>
+         <visual>
+            <origin xyz="0 0 0" rpy="0 0 0" />
+            <geometry>
+               <mesh filename="package://robots_description/meshes/Yumi/link_7.stl" />
+            </geometry>
+            <material name="Grey" />
+         </visual>
+         <collision>
+            <origin xyz="0 0 0" rpy="0 0 0" />
+            <geometry>
+               <mesh filename="package://robots_description/meshes/Yumi/coarse/link_7.stl" />
+            </geometry>
+            <material name="Grey" />
+         </collision>
+      </link>
+      <!--Extensions -->
+      <xacro:single_yumi_gazebo name="single_arm" />
+      <xacro:single_yumi_transmission name="single_arm" hardware_interface="${hardware_interface}" />
+</xacro:macro>
+  </xacro:macro>
+</robot>
+=======
+  <!-- Import all Gazebo-customization elements, including Gazebo colors -->
+  <xacro:include filename="$(find robots_description)/xacro/YumiSingleArm/single_yumi.gazebo.xacro" />
+  <!-- Import Transmissions -->
+  <xacro:include filename="$(find robots_description)/xacro/YumiSingleArm/single_yumi.transmission.xacro" />
+  <!-- some constants -->
+  <xacro:property name="joint_damping" value="0.5" />
+  <xacro:property name="max_effort" value="300" />
+  <xacro:macro name="single_yumi" params="parent hardware_interface *origin">
+    <!-- joint between external and base -->
+    <joint name="joint_0" type="fixed">
+      <xacro:insert_block name="origin"/>
+      <parent link="${parent}" />
+      <child link="single_yumi_base_link" />
+    </joint>
+    <link name="single_yumi_base_link">
+      <visual>
+        <origin xyz="0 0 0" rpy="0 0 0" />
+        <geometry>
+          <mesh filename="package://robots_description/meshes/Yumi/single_arm_base.stl" />
+        </geometry>
+        <material name="Grey" />
+      </visual>
+    </link>
+    <!-- joint between body and link_1 -->
+    <joint name="joint_1" type="revolute">
+      <parent link="single_yumi_base_link" />
+      <child link="link_1" />
+      <origin xyz="0.0 0.0 0.2048" rpy="0.0 0.0 ${PI}" />
+      <axis xyz="0 0 1" />
+      <limit lower="${-168.5 * PI / 180}" upper="${168.5 * PI / 180}"
         effort="${max_effort}" velocity="${180 * PI / 180}" />
-     <dynamics damping="${joint_damping}" />
-  </joint>
-  <link name="link_1">
-     <inertial>
+      <dynamics damping="${joint_damping}" />
+    </joint>
+    <link name="link_1">
+      <inertial>
         <origin xyz="0 -0.03 0.12" rpy="0 0 0" />
         <mass value="2" />
         <inertia ixx="0.1" ixy="0" ixz="0" iyy="0.1" iyz="0" izz="0.1" />
-     </inertial>
-     <visual>
-        <origin xyz="0 0 0" rpy="0 0 0" />
-        <geometry>
-           <mesh filename="package://robots_description/meshes/Yumi/link_1.stl" />
-        </geometry>
-        <material name="Grey" />
-     </visual>
-     <collision>
-        <origin xyz="0 0 0" rpy="0 0 0" />
-        <geometry>
-           <mesh filename="package://robots_description/meshes/Yumi/coarse/link_1.stl" />
-        </geometry>
-        <material name="Grey" />
-     </collision>
-  </link>
-  <!-- joint between link_1 and link_2 -->
-  <joint name="joint_2" type="revolute">
-     <parent link="link_1" />
-     <child link="link_2" />
-     <origin xyz="0.03 0.0 0.1" rpy="${PI / 2} 0.0 0.0" />
-     <axis xyz="0 0 1" />
-     <limit lower="${-143.5 * PI / 180}" upper="${43.5 * PI / 180}"
+      </inertial>
+      <visual>
+        <origin xyz="0 0 0" rpy="0 0 0" />
+        <geometry>
+          <mesh filename="package://robots_description/meshes/Yumi/link_1.stl" />
+        </geometry>
+        <material name="Grey" />
+      </visual>
+      <collision>
+        <origin xyz="0 0 0" rpy="0 0 0" />
+        <geometry>
+          <mesh filename="package://robots_description/meshes/Yumi/coarse/link_1.stl" />
+        </geometry>
+        <material name="Grey" />
+      </collision>
+    </link>
+    <!-- joint between link_1 and link_2 -->
+    <joint name="joint_2" type="revolute">
+      <parent link="link_1" />
+      <child link="link_2" />
+      <origin xyz="0.03 0.0 0.1" rpy="${PI / 2} 0.0 0.0" />
+      <axis xyz="0 0 1" />
+      <limit lower="${-143.5 * PI / 180}" upper="${43.5 * PI / 180}"
         effort="${max_effort}" velocity="${180 * PI / 180}" />
-     <dynamics damping="${joint_damping}" />
-  </joint>
-  <link name="link_2">
-     <inertial>
-        <origin xyz="0 0 0" rpy="0 0 0" />
-        <mass value="2" />
-        <inertia ixx="0.1" ixy="0" ixz="0" iyy="0.1" iyz="0" izz="0.1" />
-     </inertial>
-     <visual>
-        <origin xyz="0 0 0" rpy="0 0 0" />
-        <geometry>
-           <mesh filename="package://robots_description/meshes/Yumi/link_2.stl" />
-        </geometry>
-        <material name="Grey" />
-     </visual>
-     <collision>
-        <origin xyz="0 0 0" rpy="0 0 0" />
-        <geometry>
-           <mesh filename="package://robots_description/meshes/Yumi/coarse/link_2.stl" />
-        </geometry>
-        <material name="Grey" />
-     </collision>
-  </link>
-  <!-- joint between link_2 and link_3 -->
-  <joint name="joint_3" type="revolute">
-     <parent link="link_2" />
-     <child link="link_3" />
-     <origin xyz="-0.03 0.17283 0.0" rpy="${-PI / 2} 0.0 0.0" />
-     <axis xyz="0 0 1" />
-     <limit lower="${-168.5 * PI / 180}" upper="${168.5 * PI / 180}"
+      <dynamics damping="${joint_damping}" />
+    </joint>
+    <link name="link_2">
+      <inertial>
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