Commit message: Tested the abb_wrapper_control services in Gazebo

File: moveit_config/yumi_single_arm_moveit_config/config/gazebo_robot.urdf (robot description, URDF)
Before this commit: robot robot, 12 links, 11 joints
Links:
- added link grasp_link
- link single_yumi_base_link: mass None -> 2; geometry collision mesh filename=package://robots_description/meshes/Yumi/coarse/single_arm_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; visual mesh filename=package://robots_description/meshes/Yumi/single_arm_base.stl
Joints:
- removed joint gripper_joint
- removed joint gripper_joint_m
- added joint grasp_joint: type fixed, parent gripper_base, child grasp_link, origin xyz=0 0.0 0.13 rpy=0 0 0
- added joint gripper_joint_l: type prismatic, parent gripper_base, child gripper_finger_l, origin xyz=0 0.0065 0.0837 rpy=0 0 3.141592653589793, axis -1 0 0, limit lower=0 upper=0.025 effort=20 velocity=2
- added joint gripper_joint_r: type prismatic, parent gripper_base, child gripper_finger_r, origin xyz=0 -0.0065 0.0837 rpy=0 0 0, axis -1 0 0, limit lower=0 upper=0.025 effort=20 velocity=2
- joint link_7_joint: origin xyz=0 0 0.007 rpy=0 0 3.141592653589793 -> xyz=0 0.0 0.0 rpy=0 0 0

Commit message: Fixed moveit config yumi

File: moveit_config/yumi_single_arm_moveit_config/config/gazebo_robot.urdf (robot description, URDF)
Before this commit: robot robot, 12 links, 11 joints
Links:
- removed link gripper_base
- removed link gripper_finger_l
- removed link gripper_finger_r
- link single_yumi_base_link: mass None -> 0.1
Joints:
- removed joint gripper_joint
- removed joint gripper_joint_m
- removed joint link_7_joint

File: robots_description/xacro/robot.urdf.xacro (robot description, xacro)
@@ -32,12 +32,12 @@
         <!--Import
         the yumi servo gripper macro -->
-        <xacro:include filename="$(find robots_description)/Grippers/YumiServoGripper/yumi_servo_gripper.xacro" />
+        <!-- <xacro:include filename="$(find robots_description)/Grippers/YumiServoGripper/yumi_servo_gripper.xacro" /> -->
         <xacro:single_yumi parent="world" hardware_interface="${hardware_interface}">
             <origin xyz="0 0 0" rpy="0 0 0" />
         </xacro:single_yumi>
         <!-- Gripper -->
-        <xacro:yumi_servo_gripper name="gripper" parent="link_7" hardware_interface="${gripper_interface}">
+        <!-- <xacro:yumi_servo_gripper name="gripper" parent="link_7" hardware_interface="${gripper_interface}">
             <origin xyz="0 0 0.007" rpy="0 0 ${PI}" />
-        </xacro:yumi_servo_gripper>
+        </xacro:yumi_servo_gripper> -->
     </xacro:if>
 </robot>

Commit message: Possible to use yumi_single_arm in Gazebo

File: moveit_config/yumi_single_arm_moveit_config/config/gazebo_robot.urdf (robot description, URDF)
Before this commit: robot robot, 9 links, 8 joints
Links:
- added link grasp_link
- added link gripper_base, mass 0.2; collision mesh filename=package://robots_description/meshes/Yumi/gripper/coarse/bas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; visual mesh filename=package://robots_description/meshes/Yumi/gripper/base.stl
- added link gripper_finger_l, mass 0.1; collision mesh filename=package://robots_description/meshes/Yumi/gripper/coarse/fin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; visual mesh filename=package://robots_description/meshes/Yumi/gripper/finger.stl
- added link gripper_finger_r, mass 0.1; collision mesh filename=package://robots_description/meshes/Yumi/gripper/coarse/fin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; visual mesh filename=package://robots_description/meshes/Yumi/gripper/finger.stl
Joints:
- added joint grasp_joint: type fixed, parent gripper_base, child grasp_link, origin xyz=0 0.0 0.13 rpy=0 0 0
- added joint gripper_joint_l: type prismatic, parent gripper_base, child gripper_finger_l, origin xyz=0 0.0065 0.0837 rpy=0 0 3.141592653589793, axis -1 0 0, limit lower=0 upper=0.025 effort=20 velocity=2
- added joint gripper_joint_r: type prismatic, parent gripper_base, child gripper_finger_r, origin xyz=0 -0.0065 0.0837 rpy=0 0 0, axis -1 0 0, limit lower=0 upper=0.025 effort=20 velocity=2
- added joint link_7_joint: type fixed, parent link_7, child gripper_base, origin xyz=0 0.0 0.0 rpy=0 0 0

File: robots_description/xacro/robot.urdf.xacro (robot description, xacro)
@@ -30,14 +30,13 @@
         the single yumi macro -->
         <xacro:include filename="$(find robots_description)/xacro/YumiSingleArm/single_yumi.xacro" />
-        <!--Import
-        the yumi servo gripper macro -->
-        <!-- <xacro:include filename="$(find robots_description)/Grippers/YumiServoGripper/yumi_servo_gripper.xacro" /> -->
+        <!--Import the yumi servo gripper macro -->
+        <xacro:include filename="$(find robots_description)/Grippers/YumiServoGripper/yumi_servo_gripper.xacro" />
         <xacro:single_yumi parent="world" hardware_interface="${hardware_interface}">
             <origin xyz="0 0 0" rpy="0 0 0" />
         </xacro:single_yumi>
         <!-- Gripper -->
-        <!-- <xacro:yumi_servo_gripper name="gripper" parent="link_7" hardware_interface="${gripper_interface}">
+        <xacro:yumi_servo_gripper name="gripper" parent="link_7" hardware_interface="${gripper_interface}">
             <origin xyz="0 0 0.007" rpy="0 0 ${PI}" />
-        </xacro:yumi_servo_gripper> -->
+        </xacro:yumi_servo_gripper>
     </xacro:if>
 </robot>
