Commit message: Possible to simulate Gofa in Gazebo

File: gazebo_omnicore/urdf/gofa.xacro (robot description, xacro)
@@ -2,12 +2,12 @@
 <robot xmlns:xacro="http://wiki.ros.org/xacro" name="robot">
   <!-- Parameters -->
-  <arg name="name" default="yumi_single_arm" />
-  <xacro:arg name="hardware_interface" default="PositionJointInterface" />
-  <xacro:arg name="gripper_interface" default="EffortJointInterface" />
+  <arg name="name" default="gofa" />
+  <xacro:arg name="hardware_interface" default="VelocityJointInterface" />
   <xacro:arg name="base_translation" default="0" />
   <xacro:arg name="base_orientation" default="0" />
+  <xacro:arg name="child" default="flange" />
   <!-- <xacro:property name="robot" value="$(arg robot)" /> -->
   <xacro:property name="hardware_interface" value="$(arg hardware_interface)" />
-  <xacro:property name="gripper_interface" value="$(arg gripper_interface)" />
+  <xacro:property name="child" value="$(arg child)" />
   <!-- World fixed joint -->
   <link name="world" />
@@ -16,15 +16,9 @@
   <!-- Import utilities -->
   <xacro:include filename="$(find robots_description)/Util/utilities.xacro" />
-  <!--Import the single yumi macro -->
-  <xacro:include filename="$(find robots_description)/xacro/YumiSingleArm/single_yumi.xacro" />
-  <!--Import the yumi servo gripper macro -->
-  <xacro:include filename="$(find robots_description)/Grippers/YumiServoGripper/yumi_servo_gripper.xacro" />
-  <xacro:single_yumi parent="world" hardware_interface="${hardware_interface}">
+  <!--Import the gofa macro -->
+  <xacro:include filename="$(find robots_description)/xacro/Gofa/gofa.urdf.xacro" />
+  <xacro:gofa parent="world" hardware_interface="${hardware_interface}" child="${child}">
     <origin xyz="0 0 $(arg base_translation)" rpy="0 0 $(arg base_orientation)" />
-  </xacro:single_yumi>
-  <!-- Gripper -->
-  <xacro:yumi_servo_gripper name="gripper" parent="link_7" hardware_interface="${gripper_interface}">
-    <origin xyz="0 0 0.007" rpy="0 0 ${PI}" />
-  </xacro:yumi_servo_gripper>
+  </xacro:gofa>
   <!-- Loading Gazebo plugins -->
   <gazebo>

File: robots_description/xacro/Gofa/gofa.urdf.xacro (robot description, xacro)
@@ -1,8 +1,12 @@
 <?xml version="1.0"?>
 <robot xmlns:xacro="http://www.ros.org/wiki/xacro" name="gofa">
+	<!-- Import Transmissions -->
+	<xacro:include filename="$(find robots_description)/xacro/Gofa/gofa.transmission.xacro" />
 	<!-- GoFa color -->
 	<material name="gofa_color">
 		<color rgba="0.792156862745098 0.819607843137255 0.933333333333333 1"/>
 	</material>
+	<xacro:property name="joint_damping" value="0.5" />
+	<xacro:property name="max_effort" value="300" />
 	<!-- VC macro -->
 	<xacro:macro name="VC" params="suffix">
@@ -31,5 +35,5 @@
 	<xacro:arg name="6th_link_name" 	default="L6"/>
 	<!-- GoFa URDF model -->
-	<xacro:macro name="gofa" params="parent child *origin">
+	<xacro:macro name="gofa" params="parent hardware_interface child *origin">
 		<!-- Base -->
 		<joint name="${parent}_to_$(arg base_link_name)" type="fixed">
@@ -62,5 +66,6 @@
 			<child link="$(arg 1st_link_name)"/>
 			<axis xyz="0 0 1"/>
-			<limit effort="0" lower="${radians(-180)}" upper="${radians(180)}" velocity="${radians(125)}"/>
+			<limit effort="${max_effort}" lower="${radians(-180)}" upper="${radians(180)}" velocity="${radians(125)}"/>
+			<dynamics damping="${joint_damping}" />
 		</joint>
 		<!-- Link2 -->
@@ -79,5 +84,6 @@
 			<child link="$(arg 2nd_link_name)"/>
 			<axis xyz="0 1 0"/>
-			<limit effort="0" lower="${radians(-180)}" upper="${radians(180)}" velocity="${radians(125)}"/>
+			<limit effort="${max_effort}" lower="${radians(-180)}" upper="${radians(180)}" velocity="${radians(125)}"/>
+			<dynamics damping="${joint_damping}" />
 		</joint>
 		<!-- Link3 -->
@@ -96,5 +102,6 @@
 			<child link="$(arg 3rd_link_name)"/>
 			<axis xyz="0 1 0"/>
-			<limit effort="0" lower="${radians(-225)}" upper="${radians(85)}" velocity="${radians(140)}"/>
+			<limit effort="${max_effort}" lower="${radians(-225)}" upper="${radians(85)}" velocity="${radians(140)}"/>
+			<dynamics damping="${joint_damping}" />
 		</joint>
 		<!-- Link4 -->
@@ -113,5 +120,6 @@
 			<child link="$(arg 4th_link_name)"/>
 			<axis xyz="1 0 0"/>
-			<limit effort="0" lower="${radians(-180)}" upper="${radians(180)}" velocity="${radians(200)}"/>
+			<limit effort="${max_effort}" lower="${radians(-180)}" upper="${radians(180)}" velocity="${radians(200)}"/>
+			<dynamics damping="${joint_damping}" />
 		</joint>
 		<!-- Link5 -->
@@ -130,5 +138,6 @@
 			<child link="$(arg 5th_link_name)"/>
 			<axis xyz="0 1 0"/>
-			<limit effort="0" lower="${radians(-180)}" upper="${radians(180)}" velocity="${radians(200)}"/>
+			<limit effort="${max_effort}" lower="${radians(-180)}" upper="${radians(180)}" velocity="${radians(200)}"/>
+			<dynamics damping="${joint_damping}" />
 		</joint>
 		<!-- Link6 -->
@@ -147,5 +156,6 @@
 			<child link="$(arg 6th_link_name)"/>
 			<axis xyz="1 0 0"/>
-			<limit effort="0" lower="${radians(-270)}" upper="${radians(270)}" velocity="${radians(200)}"/>
+			<limit effort="${max_effort}" lower="${radians(-270)}" upper="${radians(270)}" velocity="${radians(200)}"/>
+			<dynamics damping="${joint_damping}" />
 		</joint>
 		<!-- Flange -->
@@ -157,4 +167,6 @@
 			<child link="${child}"/>
 		</joint>
+		<!--Extensions -->
+		<xacro:gofa_transmission name="gofa" hardware_interface="${hardware_interface}"/>
 	</xacro:macro>
 </robot>

File: robots_description/xacro/robot.urdf.xacro (robot description, xacro)
@@ -4,5 +4,5 @@
     <arg name="name"                    default="gofa" />
     <xacro:arg name="robot"              default="$(arg name)" />
-    <xacro:arg name="hardware_interface" default="PositionJointInterface" />
+    <xacro:arg name="hardware_interface" default="VelocityJointInterface" />
     <xacro:arg name="gripper_interface"  default="EffortJointInterface" />
     <xacro:arg name="yumi_setup"         default="default" />
@@ -16,5 +16,5 @@
     <xacro:if value="${robot == 'gofa'}">
         <xacro:include filename="$(find robots_description)/xacro/Gofa/gofa.urdf.xacro" />
-        <xacro:gofa parent="world" child="flange">
+        <xacro:gofa parent="world" hardware_interface="${hardware_interface}" child="flange">
             <origin xyz="0 0 0" rpy="0 0 0" />
         </xacro:gofa>
