Commit message: fixed naming bugs

File: omnicore_description/Grippers/YumiServoGripper/yumi_servo_gripper.xacro (robot description, xacro)
@@ -2,5 +2,5 @@
 <robot name="yumi" xmlns:xacro="http://www.ros.org/wiki/xacro">
    <!-- Import Transmissions -->
-   <xacro:include filename="$(find robots_description)/Grippers/YumiServoGripper/yumi_servo_gripper.transmission.xacro" />
+   <xacro:include filename="$(find omnicore_description)/Grippers/YumiServoGripper/yumi_servo_gripper.transmission.xacro" />
    <!-- some constants -->
    <xacro:property name="joint_damping" value="0.5" />
@@ -25,5 +25,5 @@
             <origin xyz="0 0 0" rpy="0 0 0" />
             <geometry>
-               <mesh filename="package://robots_description/meshes/Yumi/gripper/base.stl" />
+               <mesh filename="package://omnicore_description/meshes/Yumi/gripper/base.stl" />
             </geometry>
          </visual>
@@ -31,5 +31,5 @@
             <origin xyz="0 0 0" rpy="0 0 0" />
             <geometry>
-               <mesh filename="package://robots_description/meshes/Yumi/gripper/coarse/base.stl" />
+               <mesh filename="package://omnicore_description/meshes/Yumi/gripper/coarse/base.stl" />
             </geometry>
          </collision>
@@ -60,5 +60,5 @@
             <origin xyz="0 0 0" rpy="0 0 0" />
             <geometry>
-               <mesh filename="package://robots_description/meshes/Yumi/gripper/finger.stl" />
+               <mesh filename="package://omnicore_description/meshes/Yumi/gripper/finger.stl" />
             </geometry>
             <material name="Blue" />
@@ -67,5 +67,5 @@
             <origin xyz="0 0 0" rpy="0 0 0" />
             <geometry>
-               <mesh filename="package://robots_description/meshes/Yumi/gripper/coarse/finger.stl" />
+               <mesh filename="package://omnicore_description/meshes/Yumi/gripper/coarse/finger.stl" />
             </geometry>
             <material name="Blue" />
@@ -91,5 +91,5 @@
             <origin xyz="0 0 0" rpy="0 0 0" />
             <geometry>
-               <mesh filename="package://robots_description/meshes/Yumi/gripper/finger.stl" />
+               <mesh filename="package://omnicore_description/meshes/Yumi/gripper/finger.stl" />
             </geometry>
             <material name="Blue" />
@@ -98,5 +98,5 @@
             <origin xyz="0 0 0" rpy="0 0 0" />
             <geometry>
-               <mesh filename="package://robots_description/meshes/Yumi/gripper/coarse/finger.stl" />
+               <mesh filename="package://omnicore_description/meshes/Yumi/gripper/coarse/finger.stl" />
             </geometry>
             <material name="Blue" />

File: omnicore_description/xacro/Gofa/gofa.urdf.xacro (robot description, xacro)
@@ -2,5 +2,5 @@
 <robot xmlns:xacro="http://www.ros.org/wiki/xacro" name="gofa">
 	<!-- Import Transmissions -->
-	<xacro:include filename="$(find robots_description)/xacro/Gofa/gofa.transmission.xacro" />
+	<xacro:include filename="$(find omnicore_description)/xacro/Gofa/gofa.transmission.xacro" />
 	<!-- GoFa color -->
 	<material name="gofa_color">
@@ -13,5 +13,5 @@
 		<origin xyz="0 0 0" rpy="0 0 0"/>
 		<geometry>
-			<mesh filename="package://robots_description/meshes/Gofa/${suffix}.STL"/>
+			<mesh filename="package://omnicore_description/meshes/Gofa/${suffix}.STL"/>
 		</geometry>
 	</xacro:macro>

File: omnicore_description/xacro/YumiSingleArm/single_yumi.xacro (robot description, xacro)
@@ -2,7 +2,7 @@
 <robot name="single_yumi" xmlns:xacro="http://www.ros.org/wiki/xacro">
   <!-- Import all Gazebo-customization elements, including Gazebo colors -->
-  <!-- <xacro:include filename="$(find robots_description)/xacro/YumiSingleArm/single_yumi.gazebo.xacro" /> -->
+  <!-- <xacro:include filename="$(find omnicore_description)/xacro/YumiSingleArm/single_yumi.gazebo.xacro" /> -->
   <!-- Import Transmissions -->
-  <xacro:include filename="$(find robots_description)/xacro/YumiSingleArm/single_yumi.transmission.xacro" />
+  <xacro:include filename="$(find omnicore_description)/xacro/YumiSingleArm/single_yumi.transmission.xacro" />
   <!-- some constants -->
   <xacro:property name="joint_damping" value="0.5" />
@@ -19,5 +19,5 @@
         <origin xyz="0 0 0" rpy="0 0 0" />
         <geometry>
-          <mesh filename="package://robots_description/meshes/Yumi/single_arm_base.stl" />
+          <mesh filename="package://omnicore_description/meshes/Yumi/single_arm_base.stl" />
         </geometry>
         <material name="Grey" />
@@ -26,5 +26,5 @@
         <origin xyz="0 0 0" rpy="0 0 0" />
         <geometry>
-          <mesh filename="package://robots_description/meshes/Yumi/single_arm_base.stl" />
+          <mesh filename="package://omnicore_description/meshes/Yumi/single_arm_base.stl" />
         </geometry>
         <material name="Grey" />
@@ -55,12 +55,12 @@
         <origin xyz="0 0 0" rpy="0 0 0" />
         <geometry>
-          <mesh filename="package://robots_description/meshes/Yumi/link_1.stl" />
-        </geometry>
-        <material name="Grey" />
-      </visual>
-      <collision>
-        <origin xyz="0 0 0" rpy="0 0 0" />
-        <geometry>
-          <mesh filename="package://robots_description/meshes/Yumi/coarse/link_1.stl" />
+          <mesh filename="package://omnicore_description/meshes/Yumi/link_1.stl" />
+        </geometry>
+        <material name="Grey" />
+      </visual>
+      <collision>
+        <origin xyz="0 0 0" rpy="0 0 0" />
+        <geometry>
+          <mesh filename="package://omnicore_description/meshes/Yumi/coarse/link_1.stl" />
         </geometry>
         <material name="Grey" />
@@ -86,12 +86,12 @@
         <origin xyz="0 0 0" rpy="0 0 0" />
         <geometry>
-          <mesh filename="package://robots_description/meshes/Yumi/link_2.stl" />
-        </geometry>
-        <material name="Grey" />
-      </visual>
-      <collision>
-        <origin xyz="0 0 0" rpy="0 0 0" />
-        <geometry>
-          <mesh filename="package://robots_description/meshes/Yumi/coarse/link_2.stl" />
+          <mesh filename="package://omnicore_description/meshes/Yumi/link_2.stl" />
+        </geometry>
+        <material name="Grey" />
+      </visual>
+      <collision>
+        <origin xyz="0 0 0" rpy="0 0 0" />
+        <geometry>
+          <mesh filename="package://omnicore_description/meshes/Yumi/coarse/link_2.stl" />
         </geometry>
         <material name="Grey" />
@@ -117,12 +117,12 @@
         <origin xyz="0 0 0" rpy="0 0 0" />
         <geometry>
-          <mesh filename="package://robots_description/meshes/Yumi/link_3.stl" />
-        </geometry>
-        <material name="Grey" />
-      </visual>
-      <collision>
-        <origin xyz="0 0 0" rpy="0 0 0" />
-        <geometry>
-          <mesh filename="package://robots_description/meshes/Yumi/coarse/link_3.stl" />
+          <mesh filename="package://omnicore_description/meshes/Yumi/link_3.stl" />
+        </geometry>
+        <material name="Grey" />
+      </visual>
+      <collision>
+        <origin xyz="0 0 0" rpy="0 0 0" />
+        <geometry>
+          <mesh filename="package://omnicore_description/meshes/Yumi/coarse/link_3.stl" />
         </geometry>
         <material name="Grey" />
@@ -148,12 +148,12 @@
         <origin xyz="0 0 0" rpy="0 0 0" />
         <geometry>
-          <mesh filename="package://robots_description/meshes/Yumi/link_4.stl" />
-        </geometry>
-        <material name="Grey" />
-      </visual>
-      <collision>
-        <origin xyz="0 0 0" rpy="0 0 0" />
-        <geometry>
-          <mesh filename="package://robots_description/meshes/Yumi/coarse/link_4.stl" />
+          <mesh filename="package://omnicore_description/meshes/Yumi/link_4.stl" />
+        </geometry>
+        <material name="Grey" />
+      </visual>
+      <collision>
+        <origin xyz="0 0 0" rpy="0 0 0" />
+        <geometry>
+          <mesh filename="package://omnicore_description/meshes/Yumi/coarse/link_4.stl" />
         </geometry>
         <material name="Grey" />
@@ -179,12 +179,12 @@
         <origin xyz="0 0 0" rpy="0 0 0" />
         <geometry>
-          <mesh filename="package://robots_description/meshes/Yumi/link_5.stl" />
-        </geometry>
-        <material name="Grey" />
-      </visual>
-      <collision>
-        <origin xyz="0 0 0" rpy="0 0 0" />
-        <geometry>
-          <mesh filename="package://robots_description/meshes/Yumi/coarse/link_5.stl" />
+          <mesh filename="package://omnicore_description/meshes/Yumi/link_5.stl" />
+        </geometry>
+        <material name="Grey" />
+      </visual>
+      <collision>
+        <origin xyz="0 0 0" rpy="0 0 0" />
+        <geometry>
+          <mesh filename="package://omnicore_description/meshes/Yumi/coarse/link_5.stl" />
         </geometry>
         <material name="Grey" />
@@ -210,12 +210,12 @@
         <origin xyz="0 0 0" rpy="0 0 0" />
         <geometry>
-          <mesh filename="package://robots_description/meshes/Yumi/link_6.stl" />
-        </geometry>
-        <material name="Grey" />
-      </visual>
-      <collision>
-        <origin xyz="0 0 0" rpy="0 0 0" />
-        <geometry>
-          <mesh filename="package://robots_description/meshes/Yumi/coarse/link_6.stl" />
+          <mesh filename="package://omnicore_description/meshes/Yumi/link_6.stl" />
+        </geometry>
+        <material name="Grey" />
+      </visual>
+      <collision>
+        <origin xyz="0 0 0" rpy="0 0 0" />
+        <geometry>
+          <mesh filename="package://omnicore_description/meshes/Yumi/coarse/link_6.stl" />
         </geometry>
         <material name="Grey" />
@@ -241,12 +241,12 @@
         <origin xyz="0 0 0" rpy="0 0 0" />
         <geometry>
-          <mesh filename="package://robots_description/meshes/Yumi/link_7.stl" />
-        </geometry>
-        <material name="Grey" />
-      </visual>
-      <collision>
-        <origin xyz="0 0 0" rpy="0 0 0" />
-        <geometry>
-          <mesh filename="package://robots_description/meshes/Yumi/coarse/link_7.stl" />
+          <mesh filename="package://omnicore_description/meshes/Yumi/link_7.stl" />
+        </geometry>
+        <material name="Grey" />
+      </visual>
+      <collision>
+        <origin xyz="0 0 0" rpy="0 0 0" />
+        <geometry>
+          <mesh filename="package://omnicore_description/meshes/Yumi/coarse/link_7.stl" />
         </geometry>
         <material name="Grey" />

File: omnicore_description/xacro/robot.urdf.xacro (robot description, xacro)
@@ -15,5 +15,5 @@
     <!-- Gofa -->
     <xacro:if value="${robot == 'gofa'}">
-        <xacro:include filename="$(find robots_description)/xacro/Gofa/gofa.urdf.xacro" />
+        <xacro:include filename="$(find omnicore_description)/xacro/Gofa/gofa.urdf.xacro" />
         <xacro:gofa parent="world" hardware_interface="${hardware_interface}" child="flange">
             <origin xyz="0 0 0" rpy="0 0 0" />
@@ -24,12 +24,12 @@
     <xacro:if value="${robot == 'yumi_single_arm'}">
         <!-- Import Rviz colors -->
-        <xacro:include filename="$(find robots_description)/Util/materials.xacro" />
+        <xacro:include filename="$(find omnicore_description)/Util/materials.xacro" />
         <!-- Import utilities -->
-        <xacro:include filename="$(find robots_description)/Util/utilities.xacro" />
+        <xacro:include filename="$(find omnicore_description)/Util/utilities.xacro" />
         <!--Import
         the single yumi macro -->
-        <xacro:include filename="$(find robots_description)/xacro/YumiSingleArm/single_yumi.xacro" />
+        <xacro:include filename="$(find omnicore_description)/xacro/YumiSingleArm/single_yumi.xacro" />
         <!--Import the yumi servo gripper macro -->
-        <xacro:include filename="$(find robots_description)/Grippers/YumiServoGripper/yumi_servo_gripper.xacro" />
+        <xacro:include filename="$(find omnicore_description)/Grippers/YumiServoGripper/yumi_servo_gripper.xacro" />
         <xacro:single_yumi parent="world" hardware_interface="${hardware_interface}">
             <origin xyz="0 0 0" rpy="0 0 0" />

File: omnicore_gazebo/urdf/gofa.xacro (robot description, xacro)
@@ -14,9 +14,9 @@
   <link name="world" />
   <!-- Import Rviz colors -->
-  <xacro:include filename="$(find robots_description)/Util/materials.xacro" />
+  <xacro:include filename="$(find omnicore_description)/Util/materials.xacro" />
   <!-- Import utilities -->
-  <xacro:include filename="$(find robots_description)/Util/utilities.xacro" />
+  <xacro:include filename="$(find omnicore_description)/Util/utilities.xacro" />
   <!--Import the gofa macro -->
-  <xacro:include filename="$(find robots_description)/xacro/Gofa/gofa.urdf.xacro" />
+  <xacro:include filename="$(find omnicore_description)/xacro/Gofa/gofa.urdf.xacro" />
   <xacro:gofa parent="world" hardware_interface="${hardware_interface}" child="${child}">
     <origin xyz="0 0 $(arg base_translation)" rpy="0 0 $(arg base_orientation)" />

File: omnicore_gazebo/urdf/yumi_single_arm.xacro (robot description, xacro)
@@ -13,11 +13,11 @@
   <link name="world" />
   <!-- Import Rviz colors -->
-  <xacro:include filename="$(find robots_description)/Util/materials.xacro" />
+  <xacro:include filename="$(find omnicore_description)/Util/materials.xacro" />
   <!-- Import utilities -->
-  <xacro:include filename="$(find robots_description)/Util/utilities.xacro" />
+  <xacro:include filename="$(find omnicore_description)/Util/utilities.xacro" />
   <!--Import the single yumi macro -->
-  <xacro:include filename="$(find robots_description)/xacro/YumiSingleArm/single_yumi.xacro" />
+  <xacro:include filename="$(find omnicore_description)/xacro/YumiSingleArm/single_yumi.xacro" />
   <!--Import the yumi servo gripper macro -->
-  <xacro:include filename="$(find robots_description)/Grippers/YumiServoGripper/yumi_servo_gripper.xacro" />
+  <xacro:include filename="$(find omnicore_description)/Grippers/YumiServoGripper/yumi_servo_gripper.xacro" />
   <xacro:single_yumi parent="world" hardware_interface="${hardware_interface}">
     <origin xyz="0 0 $(arg base_translation)" rpy="0 0 $(arg base_orientation)" />

File: omnicore_moveit_config/gofa_moveit_config/config/gazebo_robot.urdf (robot description, URDF)
Before this commit: robot robot, 9 links, 8 joints
Links:
- link L1: geometry collision mesh filename=package://omnicore_description/meshes/Gofa/L1.STL; visual mesh filename=package://omnicore_description/meshes/Gofa/L1.STL
- link L2: geometry collision mesh filename=package://omnicore_description/meshes/Gofa/L2.STL; visual mesh filename=package://omnicore_description/meshes/Gofa/L2.STL
- link L3: geometry collision mesh filename=package://omnicore_description/meshes/Gofa/L3.STL; visual mesh filename=package://omnicore_description/meshes/Gofa/L3.STL
- link L4: geometry collision mesh filename=package://omnicore_description/meshes/Gofa/L4.STL; visual mesh filename=package://omnicore_description/meshes/Gofa/L4.STL
- link L5: geometry collision mesh filename=package://omnicore_description/meshes/Gofa/L5.STL; visual mesh filename=package://omnicore_description/meshes/Gofa/L5.STL
- link L6: geometry collision mesh filename=package://omnicore_description/meshes/Gofa/L6.STL; visual mesh filename=package://omnicore_description/meshes/Gofa/L6.STL
- link base: geometry collision mesh filename=package://omnicore_description/meshes/Gofa/base.STL; visual mesh filename=package://omnicore_description/meshes/Gofa/base.STL

File: omnicore_moveit_config/yumi_single_arm_moveit_config/config/gazebo_robot.urdf (robot description, URDF)
Before this commit: robot robot, 13 links, 12 joints
Links:
- link gripper_base: geometry collision mesh filename=package://omnicore_description/meshes/Yumi/gripper/coarse/b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; visual mesh filename=package://omnicore_description/meshes/Yumi/gripper/base.stl
- link gripper_finger_l: geometry collision mesh filename=package://omnicore_description/meshes/Yumi/gripper/coarse/f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; visual mesh filename=package://omnicore_description/meshes/Yumi/gripper/finger.s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
- link gripper_finger_r: geometry collision mesh filename=package://omnicore_description/meshes/Yumi/gripper/coarse/f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; visual mesh filename=package://omnicore_description/meshes/Yumi/gripper/finger.s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
- link link_1: geometry collision mesh filename=package://omnicore_description/meshes/Yumi/coarse/link_1.stl; visual mesh filename=package://omnicore_description/meshes/Yumi/link_1.stl
- link link_2: geometry collision mesh filename=package://omnicore_description/meshes/Yumi/coarse/link_2.stl; visual mesh filename=package://omnicore_description/meshes/Yumi/link_2.stl
- link link_3: geometry collision mesh filename=package://omnicore_description/meshes/Yumi/coarse/link_3.stl; visual mesh filename=package://omnicore_description/meshes/Yumi/link_3.stl
- link link_4: geometry collision mesh filename=package://omnicore_description/meshes/Yumi/coarse/link_4.stl; visual mesh filename=package://omnicore_description/meshes/Yumi/link_4.stl
- link link_5: geometry collision mesh filename=package://omnicore_description/meshes/Yumi/coarse/link_5.stl; visual mesh filename=package://omnicore_description/meshes/Yumi/link_5.stl
- link link_6: geometry collision mesh filename=package://omnicore_description/meshes/Yumi/coarse/link_6.stl; visual mesh filename=package://omnicore_description/meshes/Yumi/link_6.stl
- link link_7: geometry collision mesh filename=package://omnicore_description/meshes/Yumi/coarse/link_7.stl; visual mesh filename=package://omnicore_description/meshes/Yumi/link_7.stl
- link single_yumi_base_link: geometry visual mesh filename=package://omnicore_description/meshes/Yumi/single_arm_base.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
