Commit message: Added schunk gripper pkg.

File: omnicore_description/Grippers/YumiServoGripper/yumi_servo_gripper.xacro (robot description, xacro)
@@ -114,6 +114,6 @@
                <arm_name>yumi</arm_name>
                <palm_link>gripper_base</palm_link>
-               <gripper_link> gripper_finger_l </gripper_link>
-               <gripper_link> gripper_finger_r </gripper_link>
+               <gripper_link>gripper_finger_l</gripper_link>
+               <gripper_link>gripper_finger_r</gripper_link>
             </arm>
             <forces_angle_tolerance>100</forces_angle_tolerance>

File: omnicore_description/xacro/Gofa/gofa.urdf.xacro (robot description, xacro)
@@ -5,5 +5,5 @@
 	<!-- GoFa color -->
 	<material name="gofa_color">
-		<color rgba="0.792156862745098 0.819607843137255 0.933333333333333 1"/>
+		<color rgba="0.792156862745098 0.819607843137255 0.933333333333333 1" />
 	</material>
 	<xacro:property name="joint_damping" value="0.5" />
@@ -11,7 +11,7 @@
 	<!-- VC macro -->
 	<xacro:macro name="VC" params="suffix">
-		<origin xyz="0 0 0" rpy="0 0 0"/>
+		<origin xyz="0 0 0" rpy="0 0 0" />
 		<geometry>
-			<mesh filename="package://omnicore_description/meshes/Gofa/${suffix}.STL"/>
+			<mesh filename="package://omnicore_description/meshes/Gofa/${suffix}.STL" />
 		</geometry>
 	</xacro:macro>
@@ -19,53 +19,57 @@
 	<xacro:macro name="visual_plus_collision" params="v_p_c_name">
 		<visual>
-			<xacro:VC suffix="${v_p_c_name}"/>
-			<material name="gofa_color"/>
+			<xacro:VC suffix="${v_p_c_name}" />
+			<material name="gofa_color" />
 		</visual>
 		<collision>
-			<xacro:VC suffix="${v_p_c_name}"/>
+			<xacro:VC suffix="${v_p_c_name}" />
 		</collision>
 	</xacro:macro>
 	<!-- Internal link names -->
-	<xacro:arg name="base_link_name" 	default="base"/>
-	<xacro:arg name="1st_link_name" 	default="L1"/>
-	<xacro:arg name="2nd_link_name" 	default="L2"/>
-	<xacro:arg name="3rd_link_name" 	default="L3"/>
-	<xacro:arg name="4th_link_name" 	default="L4"/>
-	<xacro:arg name="5th_link_name" 	default="L5"/>
-	<xacro:arg name="6th_link_name" 	default="L6"/>
-	<xacro:arg name="flange" 	        default="flange"/>
+	<xacro:arg name="base_link_name" default="base" />
+	<xacro:arg name="1st_link_name" default="L1" />
+	<xacro:arg name="2nd_link_name" default="L2" />
+	<xacro:arg name="3rd_link_name" default="L3" />
+	<xacro:arg name="4th_link_name" default="L4" />
+	<xacro:arg name="5th_link_name" default="L5" />
+	<xacro:arg name="6th_link_name" default="L6" />
+	<xacro:arg name="flange" default="flange" />
 	<!-- GoFa URDF model -->
 	<xacro:macro name="gofa" params="parent child hardware_interface  *origin">
 		<!-- Base -->
 		<joint name="${parent}_to_${child}" type="fixed">
-			<xacro:insert_block name="origin"/>
-			<parent link="${parent}"/>
-			<child link="${child}"/>
+			<xacro:insert_block name="origin" />
+			<parent link="${parent}" />
+			<child link="${child}" />
 		</joint>
 		<link name="${child}">
 			<inertial>
-				<origin xyz="-0.0012013793465437 -0.000175191786981708 0.0862146007385352" rpy="0 0 0"/>
-				<mass value="3.50083457958494"/>
-				<inertia ixx="0.0153015257917955" ixy="-6.40155032892694E-05" ixz="-0.000276708687772683"
-						 iyy="0.0159333503953857" iyz="-3.98029144780725E-05" izz="0.0112162302268266"/>
+				<origin xyz="-0.0012013793465437 -0.000175191786981708 0.0862146007385352"
+					rpy="0 0 0" />
+				<mass value="3.50083457958494" />
+				<inertia ixx="0.0153015257917955" ixy="-6.40155032892694E-05"
+					ixz="-0.000276708687772683"
+					iyy="0.0159333503953857" iyz="-3.98029144780725E-05" izz="0.0112162302268266" />
 			</inertial>
-			<xacro:visual_plus_collision v_p_c_name="${child}"/>
+			<xacro:visual_plus_collision v_p_c_name="${child}" />
 		</link>
 		<!-- Link 1 -->
 		<link name="$(arg 1st_link_name)">
 			<inertial>
-				<origin xyz="2.08682453325091E-06 0.0103608399967513 0.0705307203199506" rpy="0 0 0"/>
-				<mass value="2.76743491139404"/>
-				<inertia ixx="0.0115158625894577" ixy="6.37197693598838E-08" ixz="5.98954393680154E-09"
-						 iyy="0.006494848329231" iyz="-0.000196668400316843" izz="0.0109446835358581"/>
+				<origin xyz="2.08682453325091E-06 0.0103608399967513 0.0705307203199506" rpy="0 0 0" />
+				<mass value="2.76743491139404" />
+				<inertia ixx="0.0115158625894577" ixy="6.37197693598838E-08"
+					ixz="5.98954393680154E-09"
+					iyy="0.006494848329231" iyz="-0.000196668400316843" izz="0.0109446835358581" />
 			</inertial>
-			<xacro:visual_plus_collision v_p_c_name="$(arg 1st_link_name)"/>
+			<xacro:visual_plus_collision v_p_c_name="$(arg 1st_link_name)" />
 		</link>
 		<joint name="J1" type="revolute">
-			<origin xyz="0 0 0.1875" rpy="0 0 0"/>
-			<parent link="${child}"/>
-			<child link="$(arg 1st_link_name)"/>
-			<axis xyz="0 0 1"/>
-			<limit effort="${max_effort}" lower="${radians(-180)}" upper="${radians(180)}" velocity="${radians(125)}"/>
+			<origin xyz="0 0 0.1875" rpy="0 0 0" />
+			<parent link="${child}" />
+			<child link="$(arg 1st_link_name)" />
+			<axis xyz="0 0 1" />
+			<limit effort="${max_effort}" lower="${radians(-180)}" upper="${radians(180)}"
+				velocity="${radians(125)}" />
 			<dynamics damping="${joint_damping}" />
 		</joint>
@@ -73,17 +77,19 @@
 		<link name="$(arg 2nd_link_name)">
 			<inertial>
-				<origin xyz="1.34018352211628E-06 -0.0500118376116071 0.222001399322246" rpy="0 0 0"/>
-				<mass value="4.28904168670464"/>
-				<inertia ixx="0.130524729873898" ixy="1.31811857134115E-07" ixz="1.99022457670482E-06"
-						 iyy="0.133278449324229" iyz="-4.48622200366709E-07" izz="0.00669457974697178"/>
+				<origin xyz="1.34018352211628E-06 -0.0500118376116071 0.222001399322246" rpy="0 0 0" />
+				<mass value="4.28904168670464" />
+				<inertia ixx="0.130524729873898" ixy="1.31811857134115E-07"
+					ixz="1.99022457670482E-06"
+					iyy="0.133278449324229" iyz="-4.48622200366709E-07" izz="0.00669457974697178" />
 			</inertial>
-			<xacro:visual_plus_collision v_p_c_name="$(arg 2nd_link_name)"/>
+			<xacro:visual_plus_collision v_p_c_name="$(arg 2nd_link_name)" />
 		</link>
 		<joint name="J2" type="revolute">
-			<origin xyz="0 -0.085 0.0775" rpy="0 0 0"/>
-			<parent link="$(arg 1st_link_name)"/>
-			<child link="$(arg 2nd_link_name)"/>
-			<axis xyz="0 1 0"/>
-			<limit effort="${max_effort}" lower="${radians(-180)}" upper="${radians(180)}" velocity="${radians(125)}"/>
+			<origin xyz="0 -0.085 0.0775" rpy="0 0 0" />
+			<parent link="$(arg 1st_link_name)" />
+			<child link="$(arg 2nd_link_name)" />
+			<axis xyz="0 1 0" />
+			<limit effort="${max_effort}" lower="${radians(-180)}" upper="${radians(180)}"
+				velocity="${radians(125)}" />
 			<dynamics damping="${joint_damping}" />
 		</joint>
@@ -91,17 +97,19 @@
 		<link name="$(arg 3rd_link_name)">
 			<inertial>
-				<origin xyz="0.0128129281453599 0.0944171780907046 0.0247427540642403" rpy="0 0 0"/>
-				<mass value="3.38333107992875"/>
-				<inertia ixx="0.0175626138728642" ixy="0.000364866179108744" ixz="-0.00318670290285352"
-						 iyy="0.0140230068919562" iyz="0.000704668055158407" izz="0.013275205067567"/>
+				<origin xyz="0.0128129281453599 0.0944171780907046 0.0247427540642403" rpy="0 0 0" />
+				<mass value="3.38333107992875" />
+				<inertia ixx="0.0175626138728642" ixy="0.000364866179108744"
+					ixz="-0.00318670290285352"
+					iyy="0.0140230068919562" iyz="0.000704668055158407" izz="0.013275205067567" />
 			</inertial>
-			<xacro:visual_plus_collision v_p_c_name="$(arg 3rd_link_name)"/>
+			<xacro:visual_plus_collision v_p_c_name="$(arg 3rd_link_name)" />
 		</link>
 		<joint name="J3" type="revolute">
-			<origin xyz="0 -0.00100000000000007 0.444" rpy="0 0 0"/>
-			<parent link="$(arg 2nd_link_name)"/>
-			<child link="$(arg 3rd_link_name)"/>
-			<axis xyz="0 1 0"/>
-			<limit effort="${max_effort}" lower="${radians(-225)}" upper="${radians(85)}" velocity="${radians(140)}"/>
+			<origin xyz="0 -0.00100000000000007 0.444" rpy="0 0 0" />
+			<parent link="$(arg 2nd_link_name)" />
+			<child link="$(arg 3rd_link_name)" />
+			<axis xyz="0 1 0" />
+			<limit effort="${max_effort}" lower="${radians(-225)}" upper="${radians(85)}"
+				velocity="${radians(140)}" />
 			<dynamics damping="${joint_damping}" />
 		</joint>
@@ -109,17 +117,19 @@
 		<link name="$(arg 4th_link_name)">
 			<inertial>
-				<origin xyz="0.160558561602322 0.041976811408979 -2.36623354021859E-07" rpy="0 0 0"/>
-				<mass value="2.77857535641324"/>
-				<inertia ixx="0.00881683095901354" ixy="-0.010746260580237" ixz="1.2899930119841E-07"
-						 iyy="0.0340754175571832" iyz="3.96362791626429E-08" izz="0.0389358932156922"/>
+				<origin xyz="0.160558561602322 0.041976811408979 -2.36623354021859E-07" rpy="0 0 0" />
+				<mass value="2.77857535641324" />
+				<inertia ixx="0.00881683095901354" ixy="-0.010746260580237"
+					ixz="1.2899930119841E-07"
+					iyy="0.0340754175571832" iyz="3.96362791626429E-08" izz="0.0389358932156922" />
 			</inertial>
-			<xacro:visual_plus_collision v_p_c_name="$(arg 4th_link_name)"/>
+			<xacro:visual_plus_collision v_p_c_name="$(arg 4th_link_name)" />
 		</link>
 		<joint name="J4" type="revolute">
-			<origin xyz="0.096 0.0860000000000001 0.11" rpy="0 0 0"/>
-			<parent link="$(arg 3rd_link_name)"/>
-			<child link="$(arg 4th_link_name)"/>
-			<axis xyz="1 0 0"/>
-			<limit effort="${max_effort}" lower="${radians(-180)}" upper="${radians(180)}" velocity="${radians(200)}"/>
+			<origin xyz="0.096 0.0860000000000001 0.11" rpy="0 0 0" />
+			<parent link="$(arg 3rd_link_name)" />
+			<child link="$(arg 4th_link_name)" />
+			<axis xyz="1 0 0" />
+			<limit effort="${max_effort}" lower="${radians(-180)}" upper="${radians(180)}"
+				velocity="${radians(200)}" />
 			<dynamics damping="${joint_damping}" />
 		</joint>
@@ -127,17 +137,19 @@
 		<link name="$(arg 5th_link_name)">
 			<inertial>
-				<origin xyz="-0.0147152361879962 -0.0785646469392633 0.0427558021601431" rpy="0 0 0"/>
-				<mass value="3.01105814739001"/>
-				<inertia ixx="0.0114597336686444" ixy="0.000180094704361231" ixz="0.00165207280226761"
-						 iyy="0.013561904467501" iyz="-0.000525272443978826" izz="0.0108480119549914"/>
+				<origin xyz="-0.0147152361879962 -0.0785646469392633 0.0427558021601431" rpy="0 0 0" />
+				<mass value="3.01105814739001" />
+				<inertia ixx="0.0114597336686444" ixy="0.000180094704361231"
+					ixz="0.00165207280226761"
+					iyy="0.013561904467501" iyz="-0.000525272443978826" izz="0.0108480119549914" />
 			</inertial>
-			<xacro:visual_plus_collision v_p_c_name="$(arg 5th_link_name)"/>
+			<xacro:visual_plus_collision v_p_c_name="$(arg 5th_link_name)" />
 		</link>
 		<joint name="J5" type="revolute">
-			<origin xyz="0.374 0.0744999999999998 0" rpy="0 0 0"/>
-			<parent link="$(arg 4th_link_name)"/>
-			<child link="$(arg 5th_link_name)"/>
-			<axis xyz="0 1 0"/>
-			<limit effort="${max_effort}" lower="${radians(-180)}" upper="${radians(180)}" velocity="${radians(200)}"/>
+			<origin xyz="0.374 0.0744999999999998 0" rpy="0 0 0" />
+			<parent link="$(arg 4th_link_name)" />
+			<child link="$(arg 5th_link_name)" />
+			<axis xyz="0 1 0" />
+			<limit effort="${max_effort}" lower="${radians(-180)}" upper="${radians(180)}"
+				velocity="${radians(200)}" />
 			<dynamics damping="${joint_damping}" />
 		</joint>
@@ -145,17 +157,21 @@
 		<link name="$(arg 6th_link_name)">
 			<inertial>
-				<origin xyz="0.0137506852604966 0.000239804131398652 -0.000341962798940165" rpy="0 0 0"/>
-				<mass value="0.146500988015653"/>
-				<inertia ixx="0.000128977630055306" ixy="-8.7622752508613E-08" ixz="1.18851551870012E-07"
-						 iyy="7.61118177829087E-05" iyz="-6.49821554399679E-07" izz="7.65022909768016E-05"/>
+				<origin xyz="0.0137506852604966 0.000239804131398652 -0.000341962798940165"
+					rpy="0 0 0" />
+				<mass value="0.146500988015653" />
+				<inertia ixx="0.000128977630055306" ixy="-8.7622752508613E-08"
+					ixz="1.18851551870012E-07"
+					iyy="7.61118177829087E-05" iyz="-6.49821554399679E-07"
+					izz="7.65022909768016E-05" />
 			</inertial>
-			<xacro:visual_plus_collision v_p_c_name="$(arg 6th_link_name)"/>
+			<xacro:visual_plus_collision v_p_c_name="$(arg 6th_link_name)" />
 		</link>
 		<joint name="J6" type="revolute">
-			<origin xyz="0.0679999999999995 -0.0744999999999998 0.0800000000000003" rpy="0 0 0"/>
-			<parent link="$(arg 5th_link_name)"/>
-			<child link="$(arg 6th_link_name)"/>
-			<axis xyz="1 0 0"/>
-			<limit effort="${max_effort}" lower="${radians(-270)}" upper="${radians(270)}" velocity="${radians(200)}"/>
+			<origin xyz="0.0679999999999995 -0.0744999999999998 0.0800000000000003" rpy="0 0 0" />
+			<parent link="$(arg 5th_link_name)" />
+			<child link="$(arg 6th_link_name)" />
+			<axis xyz="1 0 0" />
+			<limit effort="${max_effort}" lower="${radians(-270)}" upper="${radians(270)}"
+				velocity="${radians(200)}" />
 			<dynamics damping="${joint_damping}" />
 		</joint>
@@ -164,18 +180,10 @@
 		</link>
 		<joint name="$(arg 6th_link_name)_to_$(arg flange)" type="fixed">
-			<origin xyz="0.033599981 0 0" rpy="0 ${radians(90)} 0"/>
-			<parent link="$(arg 6th_link_name)"/>
-			<child link="$(arg flange)"/>
-		</joint>
-		<!-- Add fake joint for grasp_link -->
-		<link name="grasp_link">
-		</link>
-		<joint name="flange_to_grasp_link" type="fixed">
-			<origin xyz="0 0 0.05" rpy="0 0 ${pi}"/>
-			<parent link="flange"/>
-			<child link="grasp_link"/>
+			<origin xyz="0.033599981 0 0" rpy="0 ${radians(90)} 0" />
+			<parent link="$(arg 6th_link_name)" />
+			<child link="$(arg flange)" />
 		</joint>
 		<!--Extensions -->
-		<xacro:gofa_transmission name="gofa" hardware_interface="${hardware_interface}"/>
+		<xacro:gofa_transmission name="gofa" hardware_interface="${hardware_interface}" />
 	</xacro:macro>
 </robot>

File: omnicore_moveit_config/gofa_moveit_config/config/gazebo_robot.urdf (robot description, URDF)
Before this commit: robot robot, 9 links, 8 joints
Links:
- removed link base
- added link base_link_camera_stand, mass 1.0; collision box size=0.04 0.04 0.88; visual box size=0.04 0.04 0.88
- added link base_link_surface, mass 1.0; collision box size=0.6 0.4 0.1; visual box size=0.6 0.4 0.1
- added link base_link_table, mass .0; collision mesh filename=package://drims_dice_demo/meshes/Extra/table.obj scale=1.5 1 0.05; visual mesh filename=package://drims_dice_demo/meshes/Extra/table.obj scale=0.1 0.1 0.58
- added link camera_holder, mass 1.0; collision box size=0.1 0.1 0.3; visual box size=0.04 0.04 0.3
- added link ext_camera_link, mass 1e-5; visual box size=0.01 0.01 0.01
- added link finger1, mass 0.3; collision mesh filename=package://schunk_description/meshes/egk40/collision/slider.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 scale=0.001 0.001 0.001; visual mesh filename=package://schunk_description/meshes/egk40/visual/slider.dae scale=0.001 0.001 0.001
- added link finger2, mass 0.3; collision mesh filename=package://schunk_description/meshes/egk40/collision/slider.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 scale=0.001 0.001 0.001; visual mesh filename=package://schunk_description/meshes/egk40/visual/slider.dae scale=0.001 0.001 0.001
- added link gofa_base_link, mass 3.50083457958494; collision mesh filename=package://omnicore_description/meshes/Gofa/gofa_base_link.S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; visual mesh filename=package://omnicore_description/meshes/Gofa/gofa_base_link.S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
- added link gripper_body, mass 1.5; collision mesh filename=package://schunk_description/meshes/egk40/collision/egk40_b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 scale=0.001 0.001 0.001; visual mesh filename=package://schunk_description/meshes/egk40/visual/egk40_body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 scale=0.001 0.001 0.001
- added link leftfinger_body, mass 0.1; collision mesh filename=package://schunk_description/meshes/fingers/collision/flat_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 scale=0.001 0.001 0.001; visual mesh filename=package://schunk_description/meshes/fingers/visual/flat_fin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 scale=0.001 0.001 0.001
- added link rightfinger_body, mass 0.1; collision mesh filename=package://schunk_description/meshes/fingers/collision/flat_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 scale=0.001 0.001 0.001; visual mesh filename=package://schunk_description/meshes/fingers/visual/flat_fin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 scale=0.001 0.001 0.001
Joints:
- removed joint world_to_base
- added joint base_link_table_to_gofa_base_link: type fixed, parent base_link_table, child gofa_base_link, origin xyz=-0.3 0 0.627 rpy=0 0 -1.57
- added joint finger1_joint: type prismatic, parent gripper_body, child finger1, origin xyz=0.016 0.071 0.02 rpy=0 1.5707963267948966 0, limit lower=0.0 upper=0.0415 effort=1000.0 velocity=10.0
- added joint finger2_joint: type prismatic, parent gripper_body, child finger2, origin xyz=-0.016 0.071 -0.02 rpy=0 -1.5707963267948966 0, limit lower=0.0 upper=0.0415 effort=1000.0 velocity=10.0
- added joint joint_camera_holder: type fixed, parent base_link_camera_stand, child camera_holder, origin xyz=0.0 0.0 0.88 rpy=1.5707963267948966 -1.5707963267948966 0
- added joint joint_camera_link: type fixed, parent camera_holder, child ext_camera_link, origin xyz=0.0 0.0 0.4 rpy=-1.5707963267948966 0 -3.14 
- added joint joint_camera_stand_robot: type fixed, parent base_link_table, child base_link_camera_stand, origin xyz=0.0 0.4 0.65 rpy=0 0 0
- added joint joint_surface_robot: type fixed, parent gofa_base_link, child base_link_surface, origin xyz=-0.03 0.33 0.08 rpy=0 0 0
- added joint joint_table_robot: type fixed, parent world, child base_link_table, origin xyz=0 0 0 rpy=0 0 0
- added joint leftfinger_joint: type fixed, parent finger1, child leftfinger_body, origin xyz=0.0 0.012 0.0 rpy=0 0 0
- added joint parent_to_gripper: type fixed, parent flange, child gripper_body, origin xyz=0.0 0.0 0.011 rpy=1.5707963267948966 0.0 0.0
- added joint rightfinger_joint: type fixed, parent finger2, child rightfinger_body, origin xyz=0.0 0.012 0.0 rpy=0 0 0
- joint J1: limit lower=-3.141592653589793 upper=3.141592653589793 effort=0 velocity=2.181661564992912 -> lower=-3.141592653589793 upper=3.141592653589793 effort=300 velocity=2.181661564992912; parent base -> gofa_base_link
- joint J2: limit lower=-3.141592653589793 upper=3.141592653589793 effort=0 velocity=2.181661564992912 -> lower=-3.141592653589793 upper=3.141592653589793 effort=300 velocity=2.181661564992912
- joint J3: limit lower=-3.9269908169872414 upper=1.4835298641951802 effort=0 velocity=2.443460952792061 -> lower=-3.9269908169872414 upper=1.4835298641951802 effort=300 velocity=2.443460952792061
- joint J4: limit lower=-3.141592653589793 upper=3.141592653589793 effort=0 velocity=3.490658503988659 -> lower=-3.141592653589793 upper=3.141592653589793 effort=300 velocity=3.490658503988659
- joint J5: limit lower=-3.141592653589793 upper=3.141592653589793 effort=0 velocity=3.490658503988659 -> lower=-3.141592653589793 upper=3.141592653589793 effort=300 velocity=3.490658503988659
- joint J6: limit lower=-4,71239 upper=4,71239 effort=0 velocity=3.490658503988659 -> lower=-4.71238898038469 upper=4.71238898038469 effort=300 velocity=3.490658503988659
