Commit message: Minor changes.

File: schunk_ros_interface/schunk_description/urdf/egk_40_complete.xacro (robot description, xacro)
@@ -20,5 +20,5 @@
       <parent link="${parent}" />
       <child  link="grasp_link" />
-      <origin xyz="0.0 0.0 0.13" rpy="0.0 0.0 ${-pi / 2.0}" />
+      <origin xyz="0.0 0.0 0.133" rpy="0.0 0.0 ${-pi / 2.0}" />
     </joint>
     <link name="grasp_link" />

Commit message: Minor changes.

File: schunk_ros_interface/schunk_description/urdf/egk_40_complete.xacro (robot description, xacro)
@@ -20,5 +20,5 @@
       <parent link="${parent}" />
       <child  link="grasp_link" />
-      <origin xyz="0.0 0.0 0.133" rpy="0.0 0.0 ${-pi / 2.0}" />
+      <origin xyz="0.0 0.0 0.137" rpy="0.0 0.0 ${-pi / 2.0}" />
     </joint>
     <link name="grasp_link" />

Commit message: Modified grasp link frame for Schunk.

File: schunk_ros_interface/schunk_description/urdf/egk_40_complete.xacro (robot description, xacro)
@@ -20,5 +20,5 @@
       <parent link="${parent}" />
       <child  link="grasp_link" />
-      <origin xyz="0.0 0.0 0.137" rpy="0.0 0.0 ${-pi / 2.0}" />
+      <origin xyz="0.0 0.0 0.137" rpy="0.0 0.0 ${-pi / 3.0}" />
     </joint>
     <link name="grasp_link" />

Commit message: modified egk_40_complete.xacro

File: schunk_ros_interface/schunk_description/urdf/egk_40_complete.xacro (robot description, xacro)
@@ -20,5 +20,5 @@
       <parent link="${parent}" />
       <child  link="grasp_link" />
-      <origin xyz="0.0 0.0 0.137" rpy="0.0 0.0 ${-pi / 3.0}" />
+      <origin xyz="0.0 0.0 0.1375" rpy="0.0 0.0 ${-pi / 3.0}" />
     </joint>
     <link name="grasp_link" />
