Commit message: Minor changes.

File: omnicore_description/xacro/Gofa/gofa.urdf.xacro (robot description, xacro)
@@ -34,13 +34,14 @@
 	<xacro:arg name="5th_link_name" 	default="L5"/>
 	<xacro:arg name="6th_link_name" 	default="L6"/>
+	<xacro:arg name="flange" 	        default="flange"/>
 	<!-- GoFa URDF model -->
-	<xacro:macro name="gofa" params="parent hardware_interface child *origin">
+	<xacro:macro name="gofa" params="parent child hardware_interface  *origin">
 		<!-- Base -->
-		<joint name="${parent}_to_$(arg base_link_name)" type="fixed">
+		<joint name="${parent}_to_${child}" type="fixed">
 			<xacro:insert_block name="origin"/>
 			<parent link="${parent}"/>
-			<child link="$(arg base_link_name)"/>
+			<child link="${child}"/>
 		</joint>
-		<link name="$(arg base_link_name)">
+		<link name="${child}">
 			<inertial>
 				<origin xyz="-0.0012013793465437 -0.000175191786981708 0.0862146007385352" rpy="0 0 0"/>
@@ -49,5 +50,5 @@
 						 iyy="0.0159333503953857" iyz="-3.98029144780725E-05" izz="0.0112162302268266"/>
 			</inertial>
-			<xacro:visual_plus_collision v_p_c_name="$(arg base_link_name)"/>
+			<xacro:visual_plus_collision v_p_c_name="${child}"/>
 		</link>
 		<!-- Link 1 -->
@@ -63,5 +64,5 @@
 		<joint name="J1" type="revolute">
 			<origin xyz="0 0 0.1875" rpy="0 0 0"/>
-			<parent link="$(arg base_link_name)"/>
+			<parent link="${child}"/>
 			<child link="$(arg 1st_link_name)"/>
 			<axis xyz="0 0 1"/>
@@ -160,10 +161,10 @@
 		</joint>
 		<!-- Flange -->
-		<link name="${child}">
+		<link name="$(arg flange)">
 		</link>
-		<joint name="$(arg 6th_link_name)_to_${child}" type="fixed">
+		<joint name="$(arg 6th_link_name)_to_$(arg flange)" type="fixed">
 			<origin xyz="0.033599981 0 0" rpy="0 ${radians(90)} 0"/>
 			<parent link="$(arg 6th_link_name)"/>
-			<child link="${child}"/>
+			<child link="$(arg flange)"/>
 		</joint>
 		<!--Extensions -->

File: omnicore_description/xacro/YumiSingleArm/single_yumi.xacro (robot description, xacro)
@@ -8,12 +8,12 @@
   <xacro:property name="joint_damping" value="0.5" />
   <xacro:property name="max_effort" value="300" />
-  <xacro:macro name="single_yumi" params="parent hardware_interface *origin">
+  <xacro:macro name="single_yumi" params="parent child hardware_interface *origin">
     <!-- joint between external and base -->
     <joint name="joint_0" type="fixed">
       <xacro:insert_block name="origin"/>
       <parent link="${parent}" />
-      <child link="single_yumi_base_link" />
-    </joint>
-    <link name="single_yumi_base_link">
+      <child link="${child}" />
+    </joint>
+    <link name="${child}">
       <visual>
         <origin xyz="0 0 0" rpy="0 0 0" />
@@ -38,5 +38,5 @@
     <!-- joint between body and link_1 -->
     <joint name="joint_1" type="revolute">
-      <parent link="single_yumi_base_link" />
+      <parent link="${child}" />
       <child link="link_1" />
       <origin xyz="0.0 0.0 0.2048" rpy="0.0 0.0 ${PI}" />

Commit message: Add a fake grasp link to GoFa urdf.

File: omnicore_description/xacro/Gofa/gofa.urdf.xacro (robot description, xacro)
@@ -168,4 +168,12 @@
 			<child link="$(arg flange)"/>
 		</joint>
+		<!-- Add fake joint for grasp_link -->
+		<link name="grasp_link">
+		</link>
+		<joint name="flange_to_grasp_link" type="fixed">
+			<origin xyz="0 0 0.05" rpy="0 0 ${pi}"/>
+			<parent link="flange"/>
+			<child link="grasp_link"/>
+		</joint>
 		<!--Extensions -->
 		<xacro:gofa_transmission name="gofa" hardware_interface="${hardware_interface}"/>

File: omnicore_description/xacro/robot.urdf.xacro (robot description, xacro)
@@ -2,12 +2,12 @@
 <robot xmlns:xacro="http://www.ros.org/wiki/xacro" name="robot">
     <!-- Parameters -->
-    <arg name="name"                    default="gofa" />
-    <xacro:arg name="robot"              default="$(arg name)" />
+    <arg name="name" default="gofa" />
+    <xacro:arg name="robot" default="$(arg name)" />
     <xacro:arg name="hardware_interface" default="VelocityJointInterface" />
-    <xacro:arg name="gripper_interface"  default="EffortJointInterface" />
-    <xacro:arg name="yumi_setup"         default="default" />
-    <xacro:property name="robot"              value="$(arg robot)" />
+    <xacro:arg name="gripper_interface" default="EffortJointInterface" />
+    <xacro:arg name="yumi_setup" default="default" />
+    <xacro:property name="robot" value="$(arg robot)" />
     <xacro:property name="hardware_interface" value="$(arg hardware_interface)" />
-    <xacro:property name="gripper_interface"  value="$(arg gripper_interface)" />
+    <xacro:property name="gripper_interface" value="$(arg gripper_interface)" />
     <!-- World fixed joint -->
     <link name="world" />
@@ -19,8 +19,7 @@
             <origin xyz="0 0 0" rpy="0 0 0" />
         </xacro:gofa>
-        <!-- Gripper -->
     </xacro:if>
     <!-- Single Yumi -->
-    <xacro:if value="${robot == 'yumi_single_arm'}">
+    <xacro:if value="${robot == 'yumi'}">
         <!-- Import Rviz colors -->
         <xacro:include filename="$(find omnicore_description)/Util/materials.xacro" />
@@ -30,11 +29,14 @@
         the single yumi macro -->
         <xacro:include filename="$(find omnicore_description)/xacro/YumiSingleArm/single_yumi.xacro" />
-        <!--Import the yumi servo gripper macro -->
-        <xacro:include filename="$(find omnicore_description)/Grippers/YumiServoGripper/yumi_servo_gripper.xacro" />
+        <!--Import
+        the yumi servo gripper macro -->
+        <xacro:include
+            filename="$(find omnicore_description)/Grippers/YumiServoGripper/yumi_servo_gripper.xacro" />
         <xacro:single_yumi parent="world" hardware_interface="${hardware_interface}">
             <origin xyz="0 0 0" rpy="0 0 0" />
         </xacro:single_yumi>
-        <!-- Gripper -->
-        <xacro:yumi_servo_gripper name="gripper" parent="link_7" hardware_interface="${gripper_interface}">
+        <!-- YuMi Gripper -->
+        <xacro:yumi_servo_gripper name="gripper" parent="link_7"
+            hardware_interface="${gripper_interface}">
             <origin xyz="0 0 0.007" rpy="0 0 ${PI}" />
         </xacro:yumi_servo_gripper>

Commit message: fixed urdfs, fixed controller gains, regenerated moveit_config. tested in sim. to be tested on real robot

File: omnicore_description/xacro/Gofa/gofa.urdf.xacro (robot description, xacro)
@@ -27,5 +27,5 @@
 	</xacro:macro>
 	<!-- Internal link names -->
-	<xacro:arg name="base_link_name" default="base" />
+	<!--<xacro:arg name="base_link_name" default="base" /> UNUSED -->
 	<xacro:arg name="1st_link_name" default="L1" />
 	<xacro:arg name="2nd_link_name" default="L2" />

File: omnicore_description/xacro/robot.urdf.xacro (robot description, xacro)
@@ -6,5 +6,5 @@
     <xacro:arg name="hardware_interface" default="VelocityJointInterface" />
     <xacro:arg name="gripper_interface" default="EffortJointInterface" />
-    <xacro:arg name="yumi_setup" default="default" />
+    <!--<xacro:arg name="yumi_setup" default="default" /> UNUSED -->
     <xacro:property name="robot" value="$(arg robot)" />
     <xacro:property name="hardware_interface" value="$(arg hardware_interface)" />
@@ -16,10 +16,10 @@
     <xacro:if value="${robot == 'gofa'}">
         <xacro:include filename="$(find omnicore_description)/xacro/Gofa/gofa.urdf.xacro" />
-        <xacro:gofa parent="world" hardware_interface="${hardware_interface}" child="flange">
+        <xacro:gofa parent="world" hardware_interface="${hardware_interface}" child="gofa_base_link">
             <origin xyz="0 0 0" rpy="0 0 0" />
         </xacro:gofa>
     </xacro:if>
     <!-- Single Yumi -->
-    <xacro:if value="${robot == 'yumi'}">
+    <xacro:if value="${robot == 'yumi_single_arm'}">
         <!-- Import Rviz colors -->
         <xacro:include filename="$(find omnicore_description)/Util/materials.xacro" />
@@ -33,5 +33,5 @@
         <xacro:include
             filename="$(find omnicore_description)/Grippers/YumiServoGripper/yumi_servo_gripper.xacro" />
-        <xacro:single_yumi parent="world" hardware_interface="${hardware_interface}">
+        <xacro:single_yumi parent="world" hardware_interface="${hardware_interface}" child="yumi_base_link">
             <origin xyz="0 0 0" rpy="0 0 0" />
         </xacro:single_yumi>

File: omnicore_gazebo/urdf/gofa.xacro (robot description, xacro)
@@ -7,5 +7,5 @@
   <xacro:arg name="base_translation" default="0" />
   <xacro:arg name="base_orientation" default="0" />
-  <xacro:arg name="child" default="flange" />
+  <xacro:arg name="child" default="gofa_base_link" />
   <!-- <xacro:property name="robot" value="$(arg robot)" /> -->
   <xacro:property name="hardware_interface" value="$(arg hardware_interface)" />

File: omnicore_gazebo/urdf/yumi_single_arm.xacro (robot description, xacro)
@@ -7,7 +7,9 @@
   <xacro:arg name="base_translation" default="0" />
   <xacro:arg name="base_orientation" default="0" />
+  <xacro:arg name="child" default="yumi_base_link" />
   <!-- <xacro:property name="robot" value="$(arg robot)" /> -->
   <xacro:property name="hardware_interface" value="$(arg hardware_interface)" />
   <xacro:property name="gripper_interface" value="$(arg gripper_interface)" />
+  <xacro:property name="child" value="$(arg child)" />
   <!-- World fixed joint -->
   <link name="world" />
@@ -20,5 +22,5 @@
   <!--Import the yumi servo gripper macro -->
   <xacro:include filename="$(find omnicore_description)/Grippers/YumiServoGripper/yumi_servo_gripper.xacro" />
-  <xacro:single_yumi parent="world" hardware_interface="${hardware_interface}">
+  <xacro:single_yumi parent="world" hardware_interface="${hardware_interface}" child="${child}">
     <origin xyz="0 0 $(arg base_translation)" rpy="0 0 $(arg base_orientation)" />
   </xacro:single_yumi>

File: omnicore_moveit_config/yumi_single_arm_moveit_config/config/gazebo_robot.urdf (robot description, URDF)
Before this commit: robot robot, 13 links, 12 joints
Links:
- removed link single_yumi_base_link
- added link yumi_base_link, mass 0.1; visual mesh filename=package://omnicore_description/meshes/Yumi/single_arm_base.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
Joints:
- joint joint_0: child single_yumi_base_link -> yumi_base_link
- joint joint_1: limit lower=-2.940879789610445 upper=2.940879789610445 effort=300 velocity=3.141592653589793 -> lower=-2.9234264970905017 upper=2.9234264970905017 effort=300 velocity=3.141592653589793; parent single_yumi_base_link -> yumi_base_link
- joint joint_2: limit lower=-2.504547476611863 upper=0.7592182246175333 effort=300 velocity=3.141592653589793 -> lower=-2.48709418409192 upper=0.7417649320975901 effort=300 velocity=3.141592653589793
- joint joint_3: limit lower=-2.940879789610445 upper=2.940879789610445 effort=300 velocity=3.141592653589793 -> lower=-2.9234264970905017 upper=2.9234264970905017 effort=300 velocity=3.141592653589793
- joint joint_4: limit lower=-2.155481626212997 upper=1.3962634015954636 effort=300 velocity=3.141592653589793 -> lower=-2.1380283336930535 upper=1.3788101090755203 effort=300 velocity=3.141592653589793
- joint joint_5: limit lower=-5.061454830783555 upper=5.061454830783555 effort=300 velocity=6.981317007977318 -> lower=-5.044001538263612 upper=5.044001538263612 effort=300 velocity=6.981317007977318
- joint joint_6: limit lower=-1.53588974175501 upper=2.4085543677521746 effort=300 velocity=6.981317007977318 -> lower=-1.5184364492350666 upper=2.3911010752322315 effort=300 velocity=6.981317007977318
- joint joint_7: limit lower=-3.9968039870670142 upper=3.9968039870670142 effort=300 velocity=6.981317007977318 -> lower=-3.979350694547071 upper=3.979350694547071 effort=300 velocity=6.981317007977318
