Commit message: marco : added support to gofa 10 kg and gofa 12 kg. tested in simulation. to be tested on hw.

File: omnicore_description/xacro/Gofa/gofa_10.urdf.xacro (robot description, xacro)
@@ -14,5 +14,5 @@
 			<origin xyz="0 0 0" rpy="0 0 0" />
 			<geometry>
-				<mesh filename="package://omnicore_description/meshes/Gofa10/visual/${v_p_c_name}.stl"  />
+				<mesh filename="package://omnicore_description/meshes/Gofa10/visual/${v_p_c_name}.stl" />
 			</geometry>
 			<material name="gofa_color" />
@@ -21,5 +21,5 @@
 			<origin xyz="0 0 0" rpy="0 0 0" />
 			<geometry>
-				<mesh filename="package://omnicore_description/meshes/Gofa10/collision/${v_p_c_name}.stl"  />
+				<mesh filename="package://omnicore_description/meshes/Gofa10/collision/${v_p_c_name}.stl" />
 			</geometry>
 		</collision>
@@ -65,5 +65,5 @@
 		</link>
 		<joint name="J1" type="revolute">
-			<origin xyz="0 0 0.4" rpy="0 0 0"/>
+			<origin xyz="0 0.0 0.4" rpy="0 0 0"/>
 			<axis xyz="0 0 1"/>
 			<parent link="${child}" />
@@ -85,5 +85,5 @@
 		</link>
 		<joint name="J2" type="revolute">
-			<origin xyz="0 0 0" rpy="0 0 0"/>
+			<origin xyz="0.15 0 0" rpy="0 0 0"/>
 			<axis xyz="0 1 0"/>
 			<parent link="$(arg 1st_link_name)" />
