Commit message: Changed joints limits due to FlexPendant error, 1 deg

File: omnicore_description/xacro/YumiSingleArm/single_yumi.xacro (robot description, xacro)
@@ -42,5 +42,5 @@
       <origin xyz="0.0 0.0 0.2048" rpy="0.0 0.0 ${PI}" />
       <axis xyz="0 0 1" />
-      <limit lower="${-168.5 * PI / 180}" upper="${168.5 * PI / 180}"
+      <limit lower="${-167.5 * PI / 180}" upper="${167.5 * PI / 180}"
         effort="${max_effort}" velocity="${180 * PI / 180}" />
       <dynamics damping="${joint_damping}" />
@@ -73,5 +73,5 @@
       <origin xyz="0.03 0.0 0.1" rpy="${PI / 2} 0.0 0.0" />
       <axis xyz="0 0 1" />
-      <limit lower="${-143.5 * PI / 180}" upper="${43.5 * PI / 180}"
+      <limit lower="${-142.5 * PI / 180}" upper="${42.5 * PI / 180}"
         effort="${max_effort}" velocity="${180 * PI / 180}" />
       <dynamics damping="${joint_damping}" />
@@ -104,5 +104,5 @@
       <origin xyz="-0.03 0.17283 0.0" rpy="${-PI / 2} 0.0 0.0" />
       <axis xyz="0 0 1" />
-      <limit lower="${-168.5 * PI / 180}" upper="${168.5 * PI / 180}"
+      <limit lower="${-167.5 * PI / 180}" upper="${167.5 * PI / 180}"
         effort="${max_effort}" velocity="${180 * PI / 180}" />
       <dynamics damping="${joint_damping}" />
@@ -135,5 +135,5 @@
       <origin xyz="-0.04188 0.0 0.07873" rpy="${PI / 2} ${- PI / 2} 0.0" />
       <axis xyz="0 0 1" />
-      <limit lower="${-123.5 * PI / 180}" upper="${80 * PI / 180}"
+      <limit lower="${-122.5 * PI / 180}" upper="${79 * PI / 180}"
         effort="${max_effort}" velocity="${180 * PI / 180}" />
       <dynamics damping="${joint_damping}" />
@@ -166,5 +166,5 @@
       <origin xyz="0.0405 0.16461 0.0" rpy="-${PI / 2} 0.0 0.0" />
       <axis xyz="0 0 1" />
-      <limit lower="${-290 * PI / 180}" upper="${290 * PI / 180}"
+      <limit lower="${-289 * PI / 180}" upper="${289 * PI / 180}"
         effort="${max_effort}" velocity="${400 * PI / 180}" />
       <dynamics damping="${joint_damping}" />
@@ -197,5 +197,5 @@
       <origin xyz="-0.027 0 0.10039" rpy="${PI / 2} 0.0 0.0" />
       <axis xyz="0 0 1" />
-      <limit lower="${-88 * PI / 180}" upper="${138 * PI / 180}"
+      <limit lower="${-87 * PI / 180}" upper="${137 * PI / 180}"
         effort="${max_effort}" velocity="${400 * PI / 180}" />
       <dynamics damping="${joint_damping}" />
@@ -228,5 +228,5 @@
       <origin xyz="0.027 0.029 0.0" rpy="-${PI / 2} 0.0 0.0" />
       <axis xyz="0 0 1" />
-      <limit lower="${-229 * PI / 180}" upper="${229 * PI / 180}"
+      <limit lower="${-228 * PI / 180}" upper="${228 * PI / 180}"
         effort="${max_effort}" velocity="${400 * PI / 180}" />
       <dynamics damping="${joint_damping}" />

Commit message: marco : wip: started adding support for gofa 10 kg and gofa 12 kg. cleaned urdf, added collision v. visual meshes. Removed schunk pkg.

File: omnicore_description/xacro/YumiSingleArm/single_yumi.xacro (robot description, xacro)
@@ -19,15 +19,15 @@
         <origin xyz="0 0 0" rpy="0 0 0" />
         <geometry>
-          <mesh filename="package://omnicore_description/meshes/Yumi/single_arm_base.stl" />
-        </geometry>
-        <material name="Grey" />
-      </visual>
-      <!-- <collision>
-        <origin xyz="0 0 0" rpy="0 0 0" />
-        <geometry>
-          <mesh filename="package://omnicore_description/meshes/Yumi/single_arm_base.stl" />
-        </geometry>
-        <material name="Grey" />
-      </collision> -->
+          <mesh filename="package://omnicore_description/meshes/Yumi/visual/single_arm_base.stl" />
+        </geometry>
+        <material name="Grey" />
+      </visual>
+      <collision>
+        <origin xyz="0 0 0" rpy="0 0 0" />
+        <geometry>
+          <mesh filename="package://omnicore_description/meshes/Yumi/collision/single_arm_base.stl" />
+        </geometry>
+        <material name="Grey" />
+      </collision>
       <inertial>
         <origin xyz="0 0 0" rpy="0 0 0" />
@@ -55,12 +55,12 @@
         <origin xyz="0 0 0" rpy="0 0 0" />
         <geometry>
-          <mesh filename="package://omnicore_description/meshes/Yumi/link_1.stl" />
-        </geometry>
-        <material name="Grey" />
-      </visual>
-      <collision>
-        <origin xyz="0 0 0" rpy="0 0 0" />
-        <geometry>
-          <mesh filename="package://omnicore_description/meshes/Yumi/coarse/link_1.stl" />
+          <mesh filename="package://omnicore_description/meshes/Yumi/visual/link_1.stl" />
+        </geometry>
+        <material name="Grey" />
+      </visual>
+      <collision>
+        <origin xyz="0 0 0" rpy="0 0 0" />
+        <geometry>
+          <mesh filename="package://omnicore_description/meshes/Yumi/collision/link_1.stl" />
         </geometry>
         <material name="Grey" />
@@ -86,12 +86,12 @@
         <origin xyz="0 0 0" rpy="0 0 0" />
         <geometry>
-          <mesh filename="package://omnicore_description/meshes/Yumi/link_2.stl" />
-        </geometry>
-        <material name="Grey" />
-      </visual>
-      <collision>
-        <origin xyz="0 0 0" rpy="0 0 0" />
-        <geometry>
-          <mesh filename="package://omnicore_description/meshes/Yumi/coarse/link_2.stl" />
+          <mesh filename="package://omnicore_description/meshes/Yumi/visual/link_2.stl" />
+        </geometry>
+        <material name="Grey" />
+      </visual>
+      <collision>
+        <origin xyz="0 0 0" rpy="0 0 0" />
+        <geometry>
+          <mesh filename="package://omnicore_description/meshes/Yumi/collision/link_2.stl" />
         </geometry>
         <material name="Grey" />
@@ -117,12 +117,12 @@
         <origin xyz="0 0 0" rpy="0 0 0" />
         <geometry>
-          <mesh filename="package://omnicore_description/meshes/Yumi/link_3.stl" />
-        </geometry>
-        <material name="Grey" />
-      </visual>
-      <collision>
-        <origin xyz="0 0 0" rpy="0 0 0" />
-        <geometry>
-          <mesh filename="package://omnicore_description/meshes/Yumi/coarse/link_3.stl" />
+          <mesh filename="package://omnicore_description/meshes/Yumi/visual/link_3.stl" />
+        </geometry>
+        <material name="Grey" />
+      </visual>
+      <collision>
+        <origin xyz="0 0 0" rpy="0 0 0" />
+        <geometry>
+          <mesh filename="package://omnicore_description/meshes/Yumi/collision/link_3.stl" />
         </geometry>
         <material name="Grey" />
@@ -148,12 +148,12 @@
         <origin xyz="0 0 0" rpy="0 0 0" />
         <geometry>
-          <mesh filename="package://omnicore_description/meshes/Yumi/link_4.stl" />
-        </geometry>
-        <material name="Grey" />
-      </visual>
-      <collision>
-        <origin xyz="0 0 0" rpy="0 0 0" />
-        <geometry>
-          <mesh filename="package://omnicore_description/meshes/Yumi/coarse/link_4.stl" />
+          <mesh filename="package://omnicore_description/meshes/Yumi/visual/link_4.stl" />
+        </geometry>
+        <material name="Grey" />
+      </visual>
+      <collision>
+        <origin xyz="0 0 0" rpy="0 0 0" />
+        <geometry>
+          <mesh filename="package://omnicore_description/meshes/Yumi/collision/link_4.stl" />
         </geometry>
         <material name="Grey" />
@@ -179,12 +179,12 @@
         <origin xyz="0 0 0" rpy="0 0 0" />
         <geometry>
-          <mesh filename="package://omnicore_description/meshes/Yumi/link_5.stl" />
-        </geometry>
-        <material name="Grey" />
-      </visual>
-      <collision>
-        <origin xyz="0 0 0" rpy="0 0 0" />
-        <geometry>
-          <mesh filename="package://omnicore_description/meshes/Yumi/coarse/link_5.stl" />
+          <mesh filename="package://omnicore_description/meshes/Yumi/visual/link_5.stl" />
+        </geometry>
+        <material name="Grey" />
+      </visual>
+      <collision>
+        <origin xyz="0 0 0" rpy="0 0 0" />
+        <geometry>
+          <mesh filename="package://omnicore_description/meshes/Yumi/collision/link_5.stl" />
         </geometry>
         <material name="Grey" />
@@ -210,12 +210,12 @@
         <origin xyz="0 0 0" rpy="0 0 0" />
         <geometry>
-          <mesh filename="package://omnicore_description/meshes/Yumi/link_6.stl" />
-        </geometry>
-        <material name="Grey" />
-      </visual>
-      <collision>
-        <origin xyz="0 0 0" rpy="0 0 0" />
-        <geometry>
-          <mesh filename="package://omnicore_description/meshes/Yumi/coarse/link_6.stl" />
+          <mesh filename="package://omnicore_description/meshes/Yumi/visual/link_6.stl" />
+        </geometry>
+        <material name="Grey" />
+      </visual>
+      <collision>
+        <origin xyz="0 0 0" rpy="0 0 0" />
+        <geometry>
+          <mesh filename="package://omnicore_description/meshes/Yumi/collision/link_6.stl" />
         </geometry>
         <material name="Grey" />
@@ -241,12 +241,12 @@
         <origin xyz="0 0 0" rpy="0 0 0" />
         <geometry>
-          <mesh filename="package://omnicore_description/meshes/Yumi/link_7.stl" />
-        </geometry>
-        <material name="Grey" />
-      </visual>
-      <collision>
-        <origin xyz="0 0 0" rpy="0 0 0" />
-        <geometry>
-          <mesh filename="package://omnicore_description/meshes/Yumi/coarse/link_7.stl" />
+          <mesh filename="package://omnicore_description/meshes/Yumi/visual/link_7.stl" />
+        </geometry>
+        <material name="Grey" />
+      </visual>
+      <collision>
+        <origin xyz="0 0 0" rpy="0 0 0" />
+        <geometry>
+          <mesh filename="package://omnicore_description/meshes/Yumi/collision/link_7.stl" />
         </geometry>
         <material name="Grey" />

File: omnicore_description/xacro/robot.urdf.xacro (robot description, xacro)
@@ -2,5 +2,5 @@
 <robot xmlns:xacro="http://www.ros.org/wiki/xacro" name="robot">
     <!-- Parameters -->
-    <arg name="name" default="gofa" />
+    <arg name="name" default="gofa_5" />
     <xacro:arg name="robot" default="$(arg name)" />
     <xacro:arg name="hardware_interface" default="VelocityJointInterface" />
@@ -14,9 +14,23 @@
     <!-- Robot -->
     <!-- Gofa -->
-    <xacro:if value="${robot == 'gofa'}">
-        <xacro:include filename="$(find omnicore_description)/xacro/Gofa/gofa.urdf.xacro" />
-        <xacro:gofa parent="world" hardware_interface="${hardware_interface}" child="gofa_base_link">
+    <xacro:if value="${robot == 'gofa_5'}">
+        <xacro:include filename="$(find omnicore_description)/xacro/Gofa/gofa_5.urdf.xacro" />
+        <xacro:gofa5 parent="world" hardware_interface="${hardware_interface}" child="gofa_base_link">
             <origin xyz="0 0 0" rpy="0 0 0" />
-        </xacro:gofa>
+        </xacro:gofa5>
+    </xacro:if>
+    <!-- Gofa 10 kg -->
+    <xacro:if value="${robot == 'gofa_10'}">
+        <xacro:include filename="$(find omnicore_description)/xacro/Gofa/gofa_10.urdf.xacro" />
+        <xacro:gofa10 parent="world" hardware_interface="${hardware_interface}" child="gofa_base_link">
+            <origin xyz="0 0 0" rpy="0 0 0" />
+        </xacro:gofa10>
+    </xacro:if>
+    <!-- Gofa 12 kg -->
+    <xacro:if value="${robot == 'gofa_12'}">
+        <xacro:include filename="$(find omnicore_description)/xacro/Gofa/gofa_12.urdf.xacro" />
+        <xacro:gofa12 parent="world" hardware_interface="${hardware_interface}" child="gofa_base_link">
+            <origin xyz="0 0 0" rpy="0 0 0" />
+        </xacro:gofa12>
     </xacro:if>
     <!-- Single Yumi -->
@@ -32,5 +46,5 @@
         the yumi servo gripper macro -->
         <xacro:include
-            filename="$(find omnicore_description)/Grippers/YumiServoGripper/yumi_servo_gripper.xacro" />
+            filename="$(find omnicore_description)/xacro/YumiServoGripper/yumi_servo_gripper.xacro" />
         <xacro:single_yumi parent="world" hardware_interface="${hardware_interface}" child="yumi_base_link">
             <origin xyz="0 0 0" rpy="0 0 0" />

File: omnicore_gazebo/urdf/gofa.xacro (robot description, xacro)
@@ -2,5 +2,6 @@
 <robot xmlns:xacro="http://wiki.ros.org/xacro" name="robot">
   <!-- Parameters -->
-  <arg name="name" default="gofa" />
+  <xacro:arg name="robot" default="gofa" />
+  <xacro:property name="robot" value="$(arg robot)" />
   <xacro:arg name="hardware_interface" default="VelocityJointInterface" />
   <xacro:arg name="gripper_interface" default="" />
@@ -17,9 +18,26 @@
   <!-- Import utilities -->
   <xacro:include filename="$(find omnicore_description)/Util/utilities.xacro" />
-  <!--Import the gofa macro -->
-  <xacro:include filename="$(find omnicore_description)/xacro/Gofa/gofa.urdf.xacro" />
-  <xacro:gofa parent="world" hardware_interface="${hardware_interface}" child="${child}">
-    <origin xyz="0 0 $(arg base_translation)" rpy="0 0 $(arg base_orientation)" />
-  </xacro:gofa>
+  <!--Import the gofa macro
+  <xacro:include filename="$(find omnicore_description)/xacro/Gofa/gofa.urdf.xacro" />-->
+  <xacro:if value="${robot == 'gofa_5'}">
+    <xacro:include filename="$(find omnicore_description)/xacro/Gofa/gofa_5.urdf.xacro" />
+      <xacro:gofa5 parent="world" hardware_interface="${hardware_interface}" child="${child}">
+          <origin xyz="0 0 $(arg base_translation)" rpy="0 0 $(arg base_orientation)" />
+      </xacro:gofa5>
+    </xacro:if>
+    <!-- Gofa 10 kg -->
+    <xacro:if value="${robot == 'gofa_10'}">
+      <xacro:include filename="$(find omnicore_description)/xacro/Gofa/gofa_10.urdf.xacro" />
+      <xacro:gofa10 parent="world" hardware_interface="${hardware_interface}" child="${child}">
+          <origin xyz="0 0 $(arg base_translation)" rpy="0 0 $(arg base_orientation)" />
+      </xacro:gofa10>
+    </xacro:if>
+    <!-- Gofa 12 kg -->
+    <xacro:if value="${robot == 'gofa_12'}">
+      <xacro:include filename="$(find omnicore_description)/xacro/Gofa/gofa_12.urdf.xacro" />
+      <xacro:gofa12 parent="world" hardware_interface="${hardware_interface}" child="${child}">
+          <origin xyz="0 0 $(arg base_translation)" rpy="0 0 $(arg base_orientation)" />
+      </xacro:gofa12>
+    </xacro:if>
   <!-- Loading Gazebo plugins -->
   <gazebo>

File: omnicore_gazebo/urdf/yumi_single_arm.xacro (robot description, xacro)
@@ -21,5 +21,5 @@
   <xacro:include filename="$(find omnicore_description)/xacro/YumiSingleArm/single_yumi.xacro" />
   <!--Import the yumi servo gripper macro -->
-  <xacro:include filename="$(find omnicore_description)/Grippers/YumiServoGripper/yumi_servo_gripper.xacro" />
+  <xacro:include filename="$(find omnicore_description)/xacro/YumiServoGripper/yumi_servo_gripper.xacro" />
   <xacro:single_yumi parent="world" hardware_interface="${hardware_interface}" child="${child}">
     <origin xyz="0 0 $(arg base_translation)" rpy="0 0 $(arg base_orientation)" />

File: omnicore_moveit_config/yumi_single_arm_moveit_config/config/gazebo_robot.urdf (robot description, URDF)
Before this commit: robot robot, 13 links, 12 joints
Links:
- link gripper_base: geometry collision mesh filename=package://omnicore_description/meshes/YumiGripper/collision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; visual mesh filename=package://omnicore_description/meshes/YumiGripper/visual/ba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
- link gripper_finger_l: geometry collision mesh filename=package://omnicore_description/meshes/YumiGripper/collision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; visual mesh filename=package://omnicore_description/meshes/YumiGripper/visual/fi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
- link gripper_finger_r: geometry collision mesh filename=package://omnicore_description/meshes/YumiGripper/collision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; visual mesh filename=package://omnicore_description/meshes/YumiGripper/visual/fi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
- link link_1: geometry collision mesh filename=package://omnicore_description/meshes/Yumi/collision/link_1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; visual mesh filename=package://omnicore_description/meshes/Yumi/visual/link_1.stl
- link link_2: geometry collision mesh filename=package://omnicore_description/meshes/Yumi/collision/link_2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; visual mesh filename=package://omnicore_description/meshes/Yumi/visual/link_2.stl
- link link_3: geometry collision mesh filename=package://omnicore_description/meshes/Yumi/collision/link_3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; visual mesh filename=package://omnicore_description/meshes/Yumi/visual/link_3.stl
- link link_4: geometry collision mesh filename=package://omnicore_description/meshes/Yumi/collision/link_4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; visual mesh filename=package://omnicore_description/meshes/Yumi/visual/link_4.stl
- link link_5: geometry collision mesh filename=package://omnicore_description/meshes/Yumi/collision/link_5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; visual mesh filename=package://omnicore_description/meshes/Yumi/visual/link_5.stl
- link link_6: geometry collision mesh filename=package://omnicore_description/meshes/Yumi/collision/link_6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; visual mesh filename=package://omnicore_description/meshes/Yumi/visual/link_6.stl
- link link_7: geometry collision mesh filename=package://omnicore_description/meshes/Yumi/collision/link_7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; visual mesh filename=package://omnicore_description/meshes/Yumi/visual/link_7.stl
- link yumi_base_link: geometry visual mesh filename=package://omnicore_description/meshes/Yumi/visual/single_ar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
