Commit message: fixed gazebo urdf loading

File: omnicore_description/xacro/robot.urdf.xacro (robot description, xacro)
@@ -4,6 +4,6 @@
     <arg name="name" default="gofa_5" />
     <xacro:arg name="robot" default="$(arg name)" />
-    <xacro:arg name="hardware_interface" default="VelocityJointInterface" />
-    <xacro:arg name="gripper_interface" default="EffortJointInterface" />
+    <xacro:arg name="hardware_interface" default="hardware_interface/VelocityJointInterface" />
+    <xacro:arg name="gripper_interface" default="hardware_interface/EffortJointInterface" />
     <!--<xacro:arg name="yumi_setup" default="default" /> UNUSED -->
     <xacro:property name="robot" value="$(arg robot)" />

File: omnicore_gazebo/urdf/gofa.xacro (robot description, xacro)
@@ -2,6 +2,6 @@
 <robot xmlns:xacro="http://wiki.ros.org/xacro" name="robot">
   <!-- Parameters -->
-  <xacro:arg name="robot" default="gofa" />
-  <xacro:property name="robot" value="$(arg robot)" />
+  <arg name="name" default="gofa_5" />
+  <xacro:arg name="robot" default="$(arg name)" />
   <xacro:arg name="hardware_interface" default="VelocityJointInterface" />
   <xacro:arg name="gripper_interface" default="" />
@@ -10,4 +10,5 @@
   <xacro:arg name="child" default="gofa_base_link" />
   <!-- <xacro:property name="robot" value="$(arg robot)" /> -->
+  <xacro:property name="robot" value="$(arg robot)" />
   <xacro:property name="hardware_interface" value="$(arg hardware_interface)" />
   <xacro:property name="child" value="$(arg child)" />
